Commit message: added track

File: psd_ws/src/psd_vehicle_description/urdf/psd_vehicle.urdf.xacro (robot description, xacro)
@@ -14,5 +14,5 @@
   <!-- set prefix if multiple robots are used -->
   <xacro:psd_vehicle prefix="$(arg prefix)" parent="world" >
-    <origin xyz="0 0 0.19" rpy="0 0 0" />          <!-- position robot in the world -->
+    <origin xyz="0 0 0.095" rpy="0 0 0" />          <!-- position robot in the world -->
   </xacro:psd_vehicle>
   <xacro:psd_vehicle_ros2_control

File: psd_ws/src/psd_vehicle_description/urdf/psd_vehicle_macro.ros2_control.xacro (robot description, xacro)
@@ -64,12 +64,4 @@
         <param name="frame_id">tyre_RR_1</param>
       </sensor>
-      <gpio name="flange_gpios">
-        <state_interface name="digital_in_1"/>
-        <state_interface name="digital_in_2"/>
-        <command_interface name="digital_out_1"/>
-        <state_interface name="digital_out_1"/>
-        <command_interface name="digital_out_2"/>
-        <state_interface name="digital_out_2"/>
-      </gpio>
     </ros2_control>
   </xacro:macro>

File: psd_ws/src/psd_vehicle_description/urdf/psd_vehicle_macro.urdf.xacro (robot description, xacro)
@@ -28,5 +28,5 @@
         <origin xyz="0 0 0" rpy="0 0 0"/>
         <geometry>
-          <mesh filename="package://psd_vehicle_description/meshes/visual/base_link.stl" scale="0.001 0.001 0.001"/>
+          <mesh filename="$(find psd_vehicle_description)/meshes/visual/base_link.stl" scale="0.001 0.001 0.001"/>
         </geometry>
         <material name="anodized_red"/>
@@ -48,5 +48,5 @@
         <origin xyz="0.230783 -0.306869 -1.6e-05" rpy="0 0 0"/>
         <geometry>
-          <mesh filename="package://psd_vehicle_description/meshes/visual/perno_FL_1.stl" scale="0.001 0.001 0.001"/>
+          <mesh filename="$(find psd_vehicle_description)/meshes/visual/perno_FL_1.stl" scale="0.001 0.001 0.001"/>
         </geometry>
         <material name="silver"/>
@@ -68,5 +68,5 @@
         <origin xyz="0.232596 -0.307715 -1.6e-05" rpy="0 0 0"/>
         <geometry>
-          <mesh filename="package://psd_vehicle_description/meshes/visual/tyre_FL_1.stl" scale="0.001 0.001 0.001"/>
+          <mesh filename="$(find psd_vehicle_description)/meshes/visual/tyre_FL_1.stl" scale="0.001 0.001 0.001"/>
         </geometry>
         <material name="rubber_tyre"/>
@@ -78,5 +78,5 @@
         </geometry>
       </collision>
-    </link>
+    </link>z
     <link name="${prefix}perno_FR_1">
       <inertial>
@@ -88,5 +88,5 @@
         <origin xyz="-0.120217 -0.306869 -1.6e-05" rpy="0 0 0"/>
         <geometry>
-          <mesh filename="package://psd_vehicle_description/meshes/visual/perno_FR_1.stl" scale="0.001 0.001 0.001"/>
+          <mesh filename="$(find psd_vehicle_description)/meshes/visual/perno_FR_1.stl" scale="0.001 0.001 0.001"/>
         </geometry>
         <material name="silver"/>
@@ -108,5 +108,5 @@
         <origin xyz="-0.122029 -0.306024 -1.6e-05" rpy="0 0 0"/>
         <geometry>
-          <mesh filename="package://psd_vehicle_description/meshes/visual/tyre_FR_1.stl" scale="0.001 0.001 0.001"/>
+          <mesh filename="$(find psd_vehicle_description)/meshes/visual/tyre_FR_1.stl" scale="0.001 0.001 0.001"/>
         </geometry>
         <material name="rubber_tyre"/>
@@ -128,5 +128,5 @@
         <origin xyz="-0.119284 0.293131 -1.6e-05" rpy="0 0 0"/>
         <geometry>
-          <mesh filename="package://psd_vehicle_description/meshes/visual/tyre_RR_1.stl" scale="0.001 0.001 0.001"/>
+          <mesh filename="$(find psd_vehicle_description)/meshes/visual/tyre_RR_1.stl" scale="0.001 0.001 0.001"/>
         </geometry>
         <material name="rubber_tyre"/>
@@ -148,5 +148,5 @@
         <origin xyz="0.095283 0.293131 -1.6e-05" rpy="0 0 0"/>
         <geometry>
-          <mesh filename="package://psd_vehicle_description/meshes/visual/link_RL_1.stl" scale="0.001 0.001 0.001"/>
+          <mesh filename="$(find psd_vehicle_description)/meshes/visual/link_RL_1.stl" scale="0.001 0.001 0.001"/>
         </geometry>
         <material name="anodized_blue"/>
@@ -168,5 +168,5 @@
         <origin xyz="0.015283 0.293131 -1.6e-05" rpy="0 0 0"/>
         <geometry>
-          <mesh filename="package://psd_vehicle_description/meshes/visual/link_RR_1.stl" scale="0.001 0.001 0.001"/>
+          <mesh filename="$(find psd_vehicle_description)/meshes/visual/link_RR_1.stl" scale="0.001 0.001 0.001"/>
         </geometry>
         <material name="anodized_blue"/>
@@ -188,5 +188,5 @@
         <origin xyz="0.229851 0.293131 -1.6e-05" rpy="0 0 0"/>
         <geometry>
-          <mesh filename="package://psd_vehicle_description/meshes/visual/tyre_RL_1.stl" scale="0.001 0.001 0.001"/>
+          <mesh filename="$(find psd_vehicle_description)/meshes/visual/tyre_RL_1.stl" scale="0.001 0.001 0.001"/>
         </geometry>
         <material name="rubber_tyre"/>
@@ -208,5 +208,5 @@
         <origin xyz="0.095283 -0.306869 -1.6e-05" rpy="0 0 0"/>
         <geometry>
-          <mesh filename="package://psd_vehicle_description/meshes/visual/link_FL_1.stl" scale="0.001 0.001 0.001"/>
+          <mesh filename="$(find psd_vehicle_description)/meshes/visual/link_FL_1.stl" scale="0.001 0.001 0.001"/>
         </geometry>
         <material name="anodized_blue"/>
@@ -228,5 +228,5 @@
         <origin xyz="0.015283 -0.306869 -1.6e-05" rpy="0 0 0"/>
         <geometry>
-          <mesh filename="package://psd_vehicle_description/meshes/visual/link_FR_1.stl" scale="0.001 0.001 0.001"/>
+          <mesh filename="$(find psd_vehicle_description)/meshes/visual/link_FR_1.stl" scale="0.001 0.001 0.001"/>
         </geometry>
         <material name="anodized_blue"/>

Commit message: added sensor (BRINGUP NOT WORKING)

File: psd_ws/src/psd_vehicle_description/urdf/psd_vehicle.urdf.xacro (robot description, xacro)
@@ -3,8 +3,4 @@
   <!-- Use this if parameters are set from the launch file, otherwise delete -->
   <xacro:arg name="prefix" default="" />
-  <xacro:arg name="use_mock_hardware" default="false" />
-  <xacro:arg name="mock_sensor_commands" default="false" />
-  <xacro:arg name="sim_gazebo_teleop" default="false" />
-  <xacro:arg name="sim_gazebo" default="false" />
   <xacro:arg name="simulation_controllers" default="" />
   <xacro:include filename="$(find psd_vehicle_description)/urdf/psd_vehicle_macro.urdf.xacro"/>
@@ -19,50 +15,4 @@
     name="psd_vehicle"
     prefix="$(arg prefix)"
-    use_mock_hardware="$(arg use_mock_hardware)"
-    mock_sensor_commands="$(arg mock_sensor_commands)"
-    sim_gazebo="$(arg sim_gazebo)"/>
-  <xacro:if value="$(arg sim_gazebo)">
-    <!-- Gazebo plugins -->
-    <gazebo reference="world">
-    </gazebo>
-    <gazebo>
-      <plugin filename="libign_ros2_control-system.so" name="ign_ros2_control::IgnitionROS2ControlPlugin">
-        <parameters>$(arg simulation_controllers)</parameters>
-        <controller_manager_node_name>$(arg prefix)controller_manager</controller_manager_node_name>
-      </plugin>
-    </gazebo>
-  </xacro:if>
-  <xacro:if value="$(arg sim_gazebo_teleop)">
-    <!-- Gazebo plugins -->
-    <gazebo reference="world">
-    </gazebo>
-    <gazebo>
-      <plugin
-        filename="ignition-gazebo-ackermann-steering-system"
-        name="gz::sim::systems::AckermannSteering">
-        <left_joint>drive_rl</left_joint>
-        <right_joint>drive_rr</right_joint>
-        <left_steering_joint>steering_fl</left_steering_joint>
-        <right_steering_joint>steering_fr</right_steering_joint>
-        <kingpin_width>0.001</kingpin_width>
-        <steering_limit>0.5</steering_limit>
-        <wheel_base>0.6</wheel_base>
-        <wheel_separation>0.351</wheel_separation>
-        <wheel_radius>0.19</wheel_radius>
-        <min_velocity>-10</min_velocity>
-        <max_velocity>10</max_velocity>
-        <min_acceleration>-3</min_acceleration>
-        <max_acceleration>3</max_acceleration>
-      </plugin>
-      <plugin
-        filename="libignition-gazebo-diff-drive-system.so"
-        name="ignition::gazebo::systems::DiffDrive">
-        <left_joint>drive_rl</left_joint>
-        <right_joint>drive_rr</right_joint>
-        <wheel_separation>0.351</wheel_separation>
-        <wheel_radius>0.19</wheel_radius>
-        <odom_publish_frequency>10</odom_publish_frequency>
-      </plugin>
-    </gazebo>
-  </xacro:if>
+  />
 </robot>

File: psd_ws/src/psd_vehicle_description/urdf/psd_vehicle_macro.ros2_control.xacro (robot description, xacro)
@@ -3,19 +3,7 @@
   <xacro:macro name="psd_vehicle_ros2_control" params="
                 name
-                prefix
-                use_mock_hardware:=^|false
-                mock_sensor_commands:=^|false
-                sim_gazebo:=^|false"
+                prefix"
                 >
     <ros2_control name="${name}" type="system">
-      <hardware>
-        <xacro:if value="${use_mock_hardware}">
-          <plugin>mock_components/GenericSystem</plugin>
-          <param name="mock_sensor_commands">${mock_sensor_commands}</param>
-        </xacro:if>
-        <xacro:if value="${sim_gazebo}">
-          <plugin>ign_ros2_control/IgnitionSystem</plugin>
-        </xacro:if>
-      </hardware>
       <joint name="${prefix}steering_fl">
         <command_interface name="position"/>

File: psd_ws/src/psd_vehicle_description/urdf/psd_vehicle_macro.urdf.xacro (robot description, xacro)
@@ -301,4 +301,156 @@
       <child link="${prefix}link_FR_1"/>
     </joint>
+    <!-- ############## SENSORS ############## -->
+    <link name="${prefix}imu_link">
+      <visual>
+        <geometry>
+          <box size="0.1 0.1 0.1"/>
+        </geometry>
+      </visual>
+      <collision>
+        <geometry>
+          <box size="0.1 0.1 0.1"/>
+        </geometry>
+      </collision>
+    </link>
+    <joint name="${prefix}imu_joint" type="fixed">
+      <parent link="${prefix}chassis"/>
+      <child link="${prefix}imu_link"/>
+      <origin xyz="0 0 0.01"/>
+    </joint>
+    <gazebo reference="${prefix}imu_link">
+      <sensor name="imu_sensor" type="imu">
+      <plugin filename="libgazebo_ros_imu_sensor.so" name="imu_plugin">
+          <ros>
+            <namespace>/demo</namespace>
+            <remapping>~/out:=imu</remapping>
+          </ros>
+          <initial_orientation_as_reference>false</initial_orientation_as_reference>
+        </plugin>
+        <always_on>true</always_on>
+        <update_rate>100</update_rate>
+        <visualize>true</visualize>
+        <imu>
+          <angular_velocity>
+            <x>
+              <noise type="gaussian">
+                <mean>0.0</mean>
+                <stddev>2e-4</stddev>
+                <bias_mean>0.0000075</bias_mean>
+                <bias_stddev>0.0000008</bias_stddev>
+              </noise>
+            </x>
+            <y>
+              <noise type="gaussian">
+                <mean>0.0</mean>
+                <stddev>2e-4</stddev>
+                <bias_mean>0.0000075</bias_mean>
+                <bias_stddev>0.0000008</bias_stddev>
+              </noise>
+            </y>
+            <z>
+              <noise type="gaussian">
+                <mean>0.0</mean>
+                <stddev>2e-4</stddev>
+                <bias_mean>0.0000075</bias_mean>
+                <bias_stddev>0.0000008</bias_stddev>
+              </noise>
+            </z>
+          </angular_velocity>
+          <linear_acceleration>
+            <x>
+              <noise type="gaussian">
+                <mean>0.0</mean>
+                <stddev>1.7e-2</stddev>
+                <bias_mean>0.1</bias_mean>
+                <bias_stddev>0.001</bias_stddev>
+              </noise>
+            </x>
+            <y>
+              <noise type="gaussian">
+                <mean>0.0</mean>
+                <stddev>1.7e-2</stddev>
+                <bias_mean>0.1</bias_mean>
+                <bias_stddev>0.001</bias_stddev>
+              </noise>
+            </y>
+            <z>
+              <noise type="gaussian">
+                <mean>0.0</mean>
+                <stddev>1.7e-2</stddev>
+                <bias_mean>0.1</bias_mean>
+                <bias_stddev>0.001</bias_stddev>
+              </noise>
+            </z>
+          </linear_acceleration>
+        </imu>
+      </sensor>
+    </gazebo>
+    <link name="${prefix}camera_link">
+      <visual>
+        <origin xyz="0 0 0" rpy="0 0 0"/>
+        <geometry>
+          <box size="0.015 0.130 0.022"/>
+        </geometry>
+      </visual>
+      <collision>
+        <origin xyz="0 0 0" rpy="0 0 0"/>
+        <geometry>
+          <box size="0.015 0.130 0.022"/>
+        </geometry>
+      </collision>
+      <inertial>
+        <origin xyz="0 0 0" rpy="0 0 0"/>
+        <mass value="0.035"/>
+        <inertia ixx="0.001"  ixy="0"  ixz="0" iyy="0.001" iyz="0" izz="0.001" />
+      </inertial>
+    </link>
+    <joint name="${prefix}camera_joint" type="fixed">
+      <parent link="${prefix}chassis"/>
+      <child link="${prefix}camera_link"/>
+      <origin xyz="0.215 0 0.05" rpy="0 0 0"/>
+    </joint>
+    <link name="${prefix}camera_depth_frame"/>
+    <joint name="${prefix}camera_depth_joint" type="fixed">
+      <origin xyz="0 0 0" rpy="${-pi/2} 0 ${-pi/2}"/>
+      <parent link="${prefix}camera_link"/>
+      <child link="${prefix}camera_depth_frame"/>
+    </joint>
+    <gazebo reference="${prefix}camera_link">
+      <sensor name="depth_camera" type="depth">
+        <visualize>true</visualize>
+        <update_rate>30.0</update_rate>
+        <camera name="camera">
+          <horizontal_fov>1.047198</horizontal_fov>
+          <image>
+            <width>640</width>
+            <height>480</height>
+            <format>R8G8B8</format>
+          </image>
+          <clip>
+            <near>0.05</near>
+            <far>3</far>
+          </clip>
+        </camera>
+        <plugin name="depth_camera_controller" filename="libgazebo_ros_camera.so">
+          <baseline>0.2</baseline>
+          <alwaysOn>true</alwaysOn>
+          <updateRate>0.0</updateRate>
+          <frame_name>camera_depth_frame</frame_name>
+          <pointCloudCutoff>0.5</pointCloudCutoff>
+          <pointCloudCutoffMax>3.0</pointCloudCutoffMax>
+          <distortionK1>0</distortionK1>
+          <distortionK2>0</distortionK2>
+          <distortionK3>0</distortionK3>
+          <distortionT1>0</distortionT1>
+          <distortionT2>0</distortionT2>
+          <CxPrime>0</CxPrime>
+          <Cx>0</Cx>
+          <Cy>0</Cy>
+          <focalLength>0</focalLength>
+          <hackBaseline>0</hackBaseline>
+        </plugin>
+      </sensor>
+    </gazebo>
   </xacro:macro>
 </robot>
