Commit message: not functional updated urdf

File: psd_ws/src/psd_vehicle_description/urdf/materials.xacro (robot description, xacro)
@@ -45,6 +45,6 @@
       <ode>
         <epsilon>0.8</epsilon> <!-- Coefficient of restitution (elasticity) -->
-        <kp>100000000.0</kp> <!-- Contact stiffness -->
-        <kd>10.0</kd> <!-- Contact damping -->
+        <kp>1000.0</kp> <!-- Contact stiffness -->
+        <kd>10000.0</kd> <!-- Contact damping -->
       </ode>
     </elasticity>

File: psd_ws/src/psd_vehicle_description/urdf/psd_vehicle_macro.ros2_control.xacro (robot description, xacro)
@@ -13,5 +13,5 @@
       </hardware>
       <!-- steering control -->
-      <joint name="steering_fr">
+      <joint name="steering_FR">
         <command_interface name="position">
           <param name="min">"${-max_steering_angle}"</param>
@@ -22,5 +22,5 @@
         </state_interface>
       </joint>
-      <joint name="steering_fl">
+      <joint name="steering_FL">
         <command_interface name="position">
           <param name="min">"${-max_steering_angle}"</param>
@@ -32,5 +32,5 @@
       </joint>
       <!-- driving control -->
-      <joint name="drive_rl">
+      <joint name="drive_RL">
         <command_interface name="effort">
           <param name="min">"${-max_torque}"</param>
@@ -41,5 +41,5 @@
         <state_interface name="effort"/>
       </joint>
-      <joint name="drive_rr">
+      <joint name="drive_RR">
         <command_interface name="effort">
           <param name="min">"${-max_torque}"</param>
@@ -50,5 +50,5 @@
         <state_interface name="effort"/>
       </joint>
-      <joint name="drive_fl">
+      <joint name="drive_FL">
         <command_interface name="effort">
           <param name="min">"${-max_torque}"</param>
@@ -59,5 +59,5 @@
         <state_interface name="effort"/>
       </joint>
-      <joint name="drive_fr">
+      <joint name="drive_FR">
         <command_interface name="effort">
           <param name="min">"${-max_torque}"</param>

File: psd_ws/src/psd_vehicle_description/urdf/psd_vehicle_macro.urdf.xacro (robot description, xacro)
@@ -7,5 +7,7 @@
     <xacro:property name="PI" value="3.14159265359" />
     <xacro:property name="rot90" value="${90 * PI / 180}" />
+    <xacro:property name="rot180" value="${180 * PI / 180}" />
     <xacro:property name="max_steering_angle" value="${20 * PI / 180}" />
+    <xacro:property name="wheel_radius" value="0.19" />
     <!-- LINKS -->
     <!-- Chassis START-->
@@ -26,5 +28,5 @@
         <origin xyz="0 0 0" rpy="0 0 0"/>
         <geometry>
-          <mesh filename="$(find psd_vehicle_description)/stl/chassis.stl" scale="0.001 0.001 0.001"/>
+          <mesh filename="$(find psd_vehicle_description)/meshes/stl/chassis.stl" scale="0.001 0.001 0.001"/>
         </geometry>
       </collision>
@@ -120,5 +122,5 @@
         <origin xyz="0.0 0.0 0.0" rpy="0 0 0"/>
         <mass value="2.80"/>
-        <inertia ixx="0.007152" iyy="0.005137" izz="0.005138" ixy="0.0" iyz="1e-06" ixz="-0.0"/>
+        <inertia ixx="0.007152" iyy="0.005137" izz="0.005138" ixy="0.0" iyz="0.0" ixz="-0.0"/>
       </inertial>
       <visual>
@@ -127,34 +129,36 @@
           <mesh filename="$(find psd_vehicle_description)/meshes/stl/wheel.stl" scale="0.001 0.001 0.001"/>
         </geometry>
-        <material name="rubber_tyre"/>
-      </visual>
-      <collision>
+        <material name="anodized_blue"/>
+      </visual>
+      <collision>
+        <origin xyz="0.0 0.0 0.0" rpy="0 0 0"/>
+        <geometry>
+          <!-- <mesh filename="$(find psd_vehicle_description)/meshes/stl/wheel.stl" scale="0.001 0.001 0.001"/> -->
+          <cylinder radius="${wheel_radius}" length="0.08"/>
+        </geometry>
+      </collision>
+    </link>
+    <link name="wheel_FR">
+      <inertial>
+        <origin xyz="0.0 0.0 0.0" rpy="0 0 0"/>
+        <mass value="2.80"/>
+        <inertia ixx="0.007152" iyy="0.005137" izz="0.005138" ixy="0.0" iyz="0.0" ixz="-0.0"/>
+      </inertial>
+      <visual>
         <origin xyz="0.0 0.0 0.0" rpy="0 0 0"/>
         <geometry>
           <mesh filename="$(find psd_vehicle_description)/meshes/stl/wheel.stl" scale="0.001 0.001 0.001"/>
         </geometry>
-      </collision>
-    </link>
-    <link name="wheel_FR">
-      <inertial>
-        <origin xyz="0.0 0.0 0.0" rpy="0 0 0"/>
-        <mass value="2.80"/>
-        <inertia ixx="0.007152" iyy="0.005137" izz="0.005138" ixy="0.0" iyz="1e-06" ixz="-0.0"/>
-      </inertial>
-      <visual>
-        <origin xyz="0.0 0.0 0.0" rpy="0 0 0"/>
-        <geometry>
-          <mesh filename="$(find psd_vehicle_description)/meshes/stl/wheel.stl" scale="0.001 0.001 0.001"/>
-        </geometry>
-        <material name="rubber_tyre"/>
-      </visual>
-      <collision>
-        <origin xyz="0.0 0.0 0.0" rpy="0 0 0"/>
-        <geometry>
-          <mesh filename="$(find psd_vehicle_description)/meshes/stl/wheel.stl" scale="0.001 0.001 0.001"/>
-        </geometry>
-      </collision>
-    </link>
-    <link name="tyre_FL">
+        <material name="anodized_blue"/>
+      </visual>
+      <collision>
+        <origin xyz="0.0 0.0 0.0" rpy="0 0 0"/>
+        <geometry>
+          <!-- <mesh filename="$(find psd_vehicle_description)/meshes/stl/wheel.stl" scale="0.001 0.001 0.001"/> -->
+          <cylinder radius="${wheel_radius}" length="0.08"/>
+        </geometry>
+      </collision>
+    </link>
+    <!-- <link name="tyre_FL">
       <inertial>
         <origin xyz="0.0 0.0 0.0" rpy="0 0 0"/>
@@ -195,5 +199,5 @@
         </geometry>
       </collision>
-    </link>
+    </link> -->
     <!-- REAR -->
     <link name="link_RL">
@@ -241,5 +245,5 @@
         <origin xyz="0.0 0.0 0.0" rpy="0 0 0"/>
         <mass value="2.80"/>
-        <inertia ixx="0.007152" iyy="0.005137" izz="0.005138" ixy="0.0" iyz="1e-06" ixz="-0.0"/>
+        <inertia ixx="0.007152" iyy="0.005137" izz="0.005138" ixy="0.0" iyz="0.0" ixz="-0.0"/>
       </inertial>
       <visual>
@@ -248,34 +252,36 @@
           <mesh filename="$(find psd_vehicle_description)/meshes/stl/wheel.stl" scale="0.001 0.001 0.001"/>
         </geometry>
-        <material name="rubber_tyre"/>
-      </visual>
-      <collision>
+        <material name="anodized_blue"/>
+      </visual>
+      <collision>
+        <origin xyz="0.0 0.0 0.0" rpy="0 0 0"/>
+        <geometry>
+          <!-- <mesh filename="$(find psd_vehicle_description)/meshes/stl/wheel.stl" scale="0.001 0.001 0.001"/> -->
+          <cylinder radius="${wheel_radius}" length="0.08"/>
+        </geometry>
+      </collision>
+    </link>
+    <link name="wheel_RR">
+      <inertial>
+        <origin xyz="0.0 0.0 0.0" rpy="0 0 0"/>
+        <mass value="2.80"/>
+        <inertia ixx="0.007152" iyy="0.005137" izz="0.005138" ixy="0.0" iyz="0.0" ixz="-0.0"/>
+      </inertial>
+      <visual>
         <origin xyz="0.0 0.0 0.0" rpy="0 0 0"/>
         <geometry>
           <mesh filename="$(find psd_vehicle_description)/meshes/stl/wheel.stl" scale="0.001 0.001 0.001"/>
         </geometry>
-      </collision>
-    </link>
-    <link name="wheel_RR">
-      <inertial>
-        <origin xyz="0.0 0.0 0.0" rpy="0 0 0"/>
-        <mass value="2.80"/>
-        <inertia ixx="0.007152" iyy="0.005137" izz="0.005138" ixy="0.0" iyz="1e-06" ixz="-0.0"/>
-      </inertial>
-      <visual>
-        <origin xyz="0.0 0.0 0.0" rpy="0 0 0"/>
-        <geometry>
-          <mesh filename="$(find psd_vehicle_description)/meshes/stl/wheel.stl" scale="0.001 0.001 0.001"/>
-        </geometry>
-        <material name="rubber_tyre"/>
-      </visual>
-      <collision>
-        <origin xyz="0.0 0.0 0.0" rpy="0 0 0"/>
-        <geometry>
-          <mesh filename="$(find psd_vehicle_description)/meshes/stl/wheel.stl" scale="0.001 0.001 0.001"/>
-        </geometry>
-      </collision>
-    </link>
-    <link name="tyre_RL">
+        <material name="anodized_blue"/>
+      </visual>
+      <collision>
+        <origin xyz="0.0 0.0 0.0" rpy="0 0 0"/>
+        <geometry>
+          <!-- <mesh filename="$(find psd_vehicle_description)/meshes/stl/wheel.stl" scale="0.001 0.001 0.001"/> -->
+          <cylinder radius="${wheel_radius}" length="0.08"/>
+        </geometry>
+      </collision>
+    </link>
+    <!-- <link name="tyre_RL">
       <inertial>
         <origin xyz="0.0 0.0 0.0" rpy="0 0 0"/>
@@ -316,9 +322,9 @@
         </geometry>
       </collision>
-    </link>
+    </link> -->
     <!-- JOINTS -->
     <!-- SUSPENSION -->
     <joint name="suspension_FL" type="fixed">
-      <origin xyz="-0.04 0.3 0.0" rpy="0 0 0"/>
+      <origin xyz="-0.04 0.3 0.0" rpy="0 0 ${rot180}"/>
       <parent link="chassis"/>
       <child link="link_FL"/>
@@ -330,5 +336,5 @@
     </joint>
     <joint name="suspension_RL" type="fixed">
-      <origin xyz="-0.04 -0.3 0.0" rpy="0 0 0"/>
+      <origin xyz="-0.04 -0.3 0.0" rpy="0 0 ${rot180}"/>
       <parent link="chassis"/>
       <child link="link_RL"/>
@@ -341,6 +347,6 @@
     <!-- STEERING -->
     <joint name="steering_FL" type="revolute">
-      <origin xyz="-0.175 0.3 0.0" rpy="0 ${rot90} 0"/>
-      <parent link="suspension_FL"/>
+      <origin xyz="0.135 0.0 0.0" rpy="0 ${rot90} 0"/>
+      <parent link="link_FL"/>
       <child link="steering_hinge_FL"/>
       <axis xyz="0.0 0.0 1.0"/>
@@ -348,6 +354,6 @@
     </joint>
     <joint name="steering_FR" type="revolute">
-      <origin xyz="0.175 0.3 0.0" rpy="0 ${rot90} 0"/>
-      <parent link="suspension_FR"/>
+      <origin xyz="0.135 0.0 0.0" rpy="0 ${rot90} 0"/>
+      <parent link="link_FR"/>
       <child link="steering_hinge_FR"/>
       <axis xyz="0.0 0.0 1.0"/>
@@ -356,48 +362,52 @@
     <!-- DRIVE -->
     <joint name="drive_FL" type="continuous">
-      <origin xyz="-0.001813 0.000846 0.0" rpy="0 0 0"/>
+      <origin xyz="0.0 0.0 0.0" rpy="0 0 0"/>
       <parent link="steering_hinge_FL"/>
       <child link="wheel_FL"/>
-      <axis xyz="1.0 0.0 0.0"/>
+      <axis xyz="0.0 0.0 1.0"/>
+      <dynamics damping="0.2" />
     </joint>
     <joint name="drive_FR" type="continuous">
-      <origin xyz="-0.001813 0.000846 0.0" rpy="0 0 0"/>
+      <origin xyz="0.0 0.0 0.0" rpy="0 0 0"/>
       <parent link="steering_hinge_FR"/>
       <child link="wheel_FR"/>
-      <axis xyz="1.0 0.0 0.0"/>
+      <axis xyz="0.0 0.0 1.0"/>
+      <dynamics damping="0.2" />
     </joint>
     <joint name="drive_RL" type="continuous">
-      <origin xyz="-0.001813 0.000846 0.0" rpy="0 0 0"/>
-      <parent link="steering_hinge_RL"/>
+      <origin xyz="0.125 0.0 0.0" rpy="0 ${rot90} 0"/>
+      <parent link="link_RL"/>
       <child link="wheel_RL"/>
-      <axis xyz="1.0 0.0 0.0"/>
+      <axis xyz="0.0 0.0 1.0"/>
+      <dynamics damping="0.2" />
     </joint>
     <joint name="drive_RR" type="continuous">
-      <origin xyz="-0.001813 0.000846 0.0" rpy="0 0 0"/>
-      <parent link="steering_hinge_RR"/>
+      <origin xyz="0.125 0.0 0.0" rpy="0 ${rot90} 0"/>
+      <parent link="link_RR"/>
       <child link="wheel_RR"/>
-      <axis xyz="1.0 0.0 0.0"/>
+      <axis xyz="0.0 0.0 1.0"/>
+      <dynamics damping="0.2" />
     </joint>
     <!-- TYRES -->
-    <joint name="tyre_attach_FL" type="fixed">
-      <origin xyz="0.0 0.0 0.0" rpy="0 ${rot90} 0"/>
+    <!-- <joint name="tyre_attach_FL" type="fixed">
+      <origin xyz="10.0 0.0 0.0" rpy="0 0 0"/>
       <parent link="wheel_FL"/>
       <child link="tyre_FL"/>
     </joint>
     <joint name="tyre_attach_FR" type="fixed">
-      <origin xyz="0.0 0.0 0.0" rpy="0 ${rot90} 0"/>
+      <origin xyz="10.0 0.0 0.0" rpy="0 ${rot90} 0"/>
       <parent link="wheel_FR"/>
       <child link="tyre_FR"/>
     </joint>
     <joint name="tyre_attach_RL" type="fixed">
-      <origin xyz="0.0 0.0 0.0" rpy="0 ${rot90} 0"/>
+      <origin xyz="10.0 0.0 0.0" rpy="0 ${rot90} 0"/>
       <parent link="wheel_RL"/>
       <child link="tyre_RL"/>
     </joint>
     <joint name="tyre_attach_RR" type="fixed">
-      <origin xyz="0.0 0.0 0.0" rpy="0 ${rot90} 0"/>
+      <origin xyz="10.0 0.0 0.0" rpy="0 ${rot90} 0"/>
       <parent link="wheel_RR"/>
       <child link="tyre_RR"/>
-    </joint>
+    </joint> -->
   </xacro:macro>
 </robot>
