Commit message: old description file

File: psd_ws/src/psd_vehicle_description/urdf/materials.xacro (robot description, xacro)
@@ -45,6 +45,6 @@
       <ode>
         <epsilon>0.8</epsilon> <!-- Coefficient of restitution (elasticity) -->
-        <kp>1000.0</kp> <!-- Contact stiffness -->
-        <kd>10000.0</kd> <!-- Contact damping -->
+        <kp>100000000.0</kp> <!-- Contact stiffness -->
+        <kd>10.0</kd> <!-- Contact damping -->
       </ode>
     </elasticity>

File: psd_ws/src/psd_vehicle_description/urdf/psd_vehicle_macro.ros2_control.xacro (robot description, xacro)
@@ -13,5 +13,5 @@
       </hardware>
       <!-- steering control -->
-      <joint name="steering_FR">
+      <joint name="steering_fr">
         <command_interface name="position">
           <param name="min">"${-max_steering_angle}"</param>
@@ -22,5 +22,5 @@
         </state_interface>
       </joint>
-      <joint name="steering_FL">
+      <joint name="steering_fl">
         <command_interface name="position">
           <param name="min">"${-max_steering_angle}"</param>
@@ -32,5 +32,5 @@
       </joint>
       <!-- driving control -->
-      <joint name="drive_RL">
+      <joint name="drive_rl">
         <command_interface name="effort">
           <param name="min">"${-max_torque}"</param>
@@ -41,5 +41,5 @@
         <state_interface name="effort"/>
       </joint>
-      <joint name="drive_RR">
+      <joint name="drive_rr">
         <command_interface name="effort">
           <param name="min">"${-max_torque}"</param>
@@ -50,5 +50,5 @@
         <state_interface name="effort"/>
       </joint>
-      <joint name="drive_FL">
+      <joint name="drive_fl">
         <command_interface name="effort">
           <param name="min">"${-max_torque}"</param>
@@ -59,5 +59,5 @@
         <state_interface name="effort"/>
       </joint>
-      <joint name="drive_FR">
+      <joint name="drive_fr">
         <command_interface name="effort">
           <param name="min">"${-max_torque}"</param>

File: psd_ws/src/psd_vehicle_description/urdf/psd_vehicle_macro.urdf.xacro (robot description, xacro)
@@ -5,21 +5,16 @@
   <!-- start vehicle description -->
   <xacro:macro name="psd_vehicle" params="parent *origin">
-    <xacro:property name="PI" value="3.14159265359" />
-    <xacro:property name="rot90" value="${90 * PI / 180}" />
-    <xacro:property name="rot180" value="${180 * PI / 180}" />
-    <xacro:property name="max_steering_angle" value="${20 * PI / 180}" />
-    <xacro:property name="wheel_radius" value="0.19" />
     <!-- LINKS -->
     <!-- Chassis START-->
     <link name="chassis">
       <inertial>
-        <origin xyz="0.0 0.0 0.0" rpy="0 0 0"/>
-        <mass value="10.0"/>
-        <inertia ixx="0.354236" iyy="0.082009" izz="0.401568" ixy="0.0" iyz="0.0" ixz="0.0"/>
+        <origin xyz="-0.055282024534886974 0.006459558608433099 1.621642854614675e-05" rpy="0 0 0"/>
+        <mass value="7.077984465449566"/>
+        <inertia ixx="0.233109" iyy="0.053798" izz="0.264742" ixy="-0.0" iyz="-0.0" ixz="-0.0"/>
       </inertial>
       <visual>
         <origin xyz="0 0 0" rpy="0 0 0"/>
         <geometry>
-          <mesh filename="$(find psd_vehicle_description)/meshes/stl/chassis.stl" scale="0.001 0.001 0.001"/>
+          <mesh filename="$(find psd_vehicle_description)/meshes/visual/base_link.stl" scale="0.001 0.001 0.001"/>
         </geometry>
         <material name="anodized_red"/>
@@ -28,9 +23,8 @@
         <origin xyz="0 0 0" rpy="0 0 0"/>
         <geometry>
-          <mesh filename="$(find psd_vehicle_description)/meshes/stl/chassis.stl" scale="0.001 0.001 0.001"/>
-        </geometry>
-      </collision>
-    </link>
-    <!-- FRONT -->
+          <mesh filename="$(find psd_vehicle_description)/meshes/collision/base_link.stl" scale="0.001 0.001 0.001"/>
+        </geometry>
+      </collision>
+    </link>
     <joint name="world_joint" type="fixed">
       <xacro:insert_block name="origin" />
@@ -38,376 +32,263 @@
       <child link="chassis" />
     </joint>
-    <link name="link_FL">
-      <inertial>
-        <origin xyz="0.0 0.0 0.0" rpy="0 0 0"/>
-        <mass value="0.270"/>
-        <inertia ixx="0.000189" iyy="0.000409" izz="0.000593" ixy="0.0" iyz="0.0" ixz="-0.0"/>
-      </inertial>
-      <visual>
-        <origin xyz="0.0 0.0 0.0" rpy="0 0 0"/>
-        <geometry>
-          <mesh filename="$(find psd_vehicle_description)/meshes/stl/suspension.stl" scale="0.001 0.001 0.001"/>
-        </geometry>
-        <material name="anodized_blue"/>
-      </visual>
-      <collision>
-        <origin xyz="0.0 0.0 0.0" rpy="0 0 0"/>
-        <geometry>
-          <mesh filename="$(find psd_vehicle_description)/meshes/stl/suspension.stl" scale="0.001 0.001 0.001"/>
-        </geometry>
-      </collision>
-    </link>
-    <link name="link_FR">
-      <inertial>
-        <origin xyz="0.0 0.0 0.0" rpy="0 0 0"/>
-        <mass value="0.270"/>
-        <inertia ixx="0.000189" iyy="0.000409" izz="0.000593" ixy="0.0" iyz="0.0" ixz="-0.0"/>
-      </inertial>
-      <visual>
-        <origin xyz="0.0 0.0 0.0" rpy="0 0 0"/>
-        <geometry>
-          <mesh filename="$(find psd_vehicle_description)/meshes/stl/suspension.stl" scale="0.001 0.001 0.001"/>
-        </geometry>
-        <material name="anodized_blue"/>
-      </visual>
-      <collision>
-        <origin xyz="0.0 0.0 0.0" rpy="0 0 0"/>
-        <geometry>
-          <mesh filename="$(find psd_vehicle_description)/meshes/stl/suspension.stl" scale="0.001 0.001 0.001"/>
-        </geometry>
-      </collision>
-    </link>
-    <link name="steering_hinge_FL">
-      <inertial>
-        <origin xyz="0.0 0.0 0.0" rpy="0 0 0"/>
-        <mass value="0.155"/>
+    <link name="perno_FL_1">
+      <inertial>
+        <origin xyz="-0.000906687358749575 0.00042296243032097225 2.1642838935455414e-07" rpy="0 0 0"/>
+        <mass value="0.00011097676048806171"/>
         <inertia ixx="0.0" iyy="0.0" izz="0.0" ixy="-0.0" iyz="0.0" ixz="-0.0"/>
       </inertial>
       <visual>
-        <origin xyz="0.0 0.0 0.0" rpy="0 0 0"/>
-        <geometry>
-          <mesh filename="$(find psd_vehicle_description)/meshes/stl/steering_hinge.stl" scale="0.001 0.001 0.001"/>
+        <origin xyz="0.230783 -0.306869 -1.6e-05" rpy="0 0 0"/>
+        <geometry>
+          <mesh filename="$(find psd_vehicle_description)/meshes/visual/perno_FL_1.stl" scale="0.001 0.001 0.001"/>
         </geometry>
         <material name="silver"/>
       </visual>
       <collision>
-        <origin xyz="0.0 0.0 0.0" rpy="0 0 0"/>
-        <geometry>
-          <mesh filename="$(find psd_vehicle_description)/meshes/stl/steering_hinge.stl" scale="0.001 0.001 0.001"/>
-        </geometry>
-      </collision>
-    </link>
-    <link name="steering_hinge_FR">
-      <inertial>
-        <origin xyz="0.0 0.0 0.0" rpy="0 0 0"/>
-        <mass value="0.155"/>
-        <inertia ixx="0.0" iyy="0.0" izz="0.0" ixy="-0.0" iyz="0.0" ixz="-0.0"/>
-      </inertial>
-      <visual>
-        <origin xyz="0.0 0.0 0.0" rpy="0 0 0"/>
-        <geometry>
-          <mesh filename="$(find psd_vehicle_description)/meshes/stl/steering_hinge.stl" scale="0.001 0.001 0.001"/>
+        <origin xyz="0.230783 -0.306869 -1.6e-05" rpy="0 0 0"/>
+        <geometry>
+          <mesh filename="$(find psd_vehicle_description)/meshes/collision/perno_FL_1.stl" scale="0.001 0.001 0.001"/>
+        </geometry>
+      </collision>
+    </link>
+    <link name="tyre_FL_1">
+      <inertial>
+        <origin xyz="-0.03851807609484373 0.017960856816041648 2.1642854673904234e-07" rpy="0 0 0"/>
+        <mass value="0.1944554118066591"/>
+        <inertia ixx="0.001191" iyy="0.000933" izz="0.000861" ixy="-0.000154" iyz="0.0" ixz="0.0"/>
+      </inertial>
+      <visual>
+        <origin xyz="0.232596 -0.307715 -1.6e-05" rpy="0 0 0"/>
+        <geometry>
+          <mesh filename="$(find psd_vehicle_description)/meshes/visual/tyre_FL_1.stl" scale="0.001 0.001 0.001"/>
+        </geometry>
+        <material name="anodized_blue"/>
+      </visual>
+      <collision>
+        <origin xyz="0.232596 -0.307715 -1.6e-05" rpy="0 0 0"/>
+        <geometry>
+          <mesh filename="$(find psd_vehicle_description)/meshes/collision/tyre_FL_1.stl" scale="0.001 0.001 0.001"/>
+        </geometry>
+      </collision>
+    </link>z
+    <link name="perno_FR_1">
+      <inertial>
+        <origin xyz="0.000905928215323884 -0.0004222740931605351 2.1642839664261197e-07" rpy="0 0 0"/>
+        <mass value="0.0001109767604880609"/>
+        <inertia ixx="0.0" iyy="0.0" izz="0.0" ixy="-0.0" iyz="-0.0" ixz="0.0"/>
+      </inertial>
+      <visual>
+        <origin xyz="-0.120217 -0.306869 -1.6e-05" rpy="0 0 0"/>
+        <geometry>
+          <mesh filename="$(find psd_vehicle_description)/meshes/visual/perno_FR_1.stl" scale="0.001 0.001 0.001"/>
         </geometry>
         <material name="silver"/>
       </visual>
       <collision>
-        <origin xyz="0.0 0.0 0.0" rpy="0 0 0"/>
-        <geometry>
-          <mesh filename="$(find psd_vehicle_description)/meshes/stl/steering_hinge.stl" scale="0.001 0.001 0.001"/>
-        </geometry>
-      </collision>
-    </link>
-    <link name="wheel_FL">
-      <inertial>
-        <origin xyz="0.0 0.0 0.0" rpy="0 0 0"/>
-        <mass value="2.80"/>
-        <inertia ixx="0.007152" iyy="0.005137" izz="0.005138" ixy="0.0" iyz="0.0" ixz="-0.0"/>
-      </inertial>
-      <visual>
-        <origin xyz="0.0 0.0 0.0" rpy="0 0 0"/>
-        <geometry>
-          <mesh filename="$(find psd_vehicle_description)/meshes/stl/wheel.stl" scale="0.001 0.001 0.001"/>
-        </geometry>
-        <material name="anodized_blue"/>
-      </visual>
-      <collision>
-        <origin xyz="0.0 0.0 0.0" rpy="0 0 0"/>
-        <geometry>
-          <!-- <mesh filename="$(find psd_vehicle_description)/meshes/stl/wheel.stl" scale="0.001 0.001 0.001"/> -->
-          <cylinder radius="${wheel_radius}" length="0.08"/>
-        </geometry>
-      </collision>
-    </link>
-    <link name="wheel_FR">
-      <inertial>
-        <origin xyz="0.0 0.0 0.0" rpy="0 0 0"/>
-        <mass value="2.80"/>
-        <inertia ixx="0.007152" iyy="0.005137" izz="0.005138" ixy="0.0" iyz="0.0" ixz="-0.0"/>
-      </inertial>
-      <visual>
-        <origin xyz="0.0 0.0 0.0" rpy="0 0 0"/>
-        <geometry>
-          <mesh filename="$(find psd_vehicle_description)/meshes/stl/wheel.stl" scale="0.001 0.001 0.001"/>
-        </geometry>
-        <material name="anodized_blue"/>
-      </visual>
-      <collision>
-        <origin xyz="0.0 0.0 0.0" rpy="0 0 0"/>
-        <geometry>
-          <!-- <mesh filename="$(find psd_vehicle_description)/meshes/stl/wheel.stl" scale="0.001 0.001 0.001"/> -->
-          <cylinder radius="${wheel_radius}" length="0.08"/>
-        </geometry>
-      </collision>
-    </link>
-    <!-- <link name="tyre_FL">
-      <inertial>
-        <origin xyz="0.0 0.0 0.0" rpy="0 0 0"/>
-        <mass value="4.40"/>
-        <inertia ixx="0.029818" iyy="0.017591" izz="0.017591" ixy="-0.0" iyz="0.0" ixz="0.0"/>
-      </inertial>
-      <visual>
-        <origin xyz="0.0 0.0 0.0" rpy="0 0 0"/>
-        <geometry>
-          <mesh filename="$(find psd_vehicle_description)/meshes/stl/tyre.stl" scale="0.001 0.001 0.001"/>
-        </geometry>
-        <material name="rubber_tyre"/>
-      </visual>
-      <collision>
-        <origin xyz="0.0 0.0 0.0" rpy="0 0 0"/>
-        <geometry>
-          <mesh filename="$(find psd_vehicle_description)/meshes/stl/tyre.stl" scale="0.001 0.001 0.001"/>
-        </geometry>
-      </collision>
-    </link>
-    <link name="tyre_FR">
-      <inertial>
-        <origin xyz="0.0 0.0 0.0" rpy="0 0 0"/>
-        <mass value="4.40"/>
-        <inertia ixx="0.029818" iyy="0.017591" izz="0.017591" ixy="-0.0" iyz="0.0" ixz="0.0"/>
-      </inertial>
-      <visual>
-        <origin xyz="0.0 0.0 0.0" rpy="0 0 0"/>
-        <geometry>
-          <mesh filename="$(find psd_vehicle_description)/meshes/stl/tyre.stl" scale="0.001 0.001 0.001"/>
-        </geometry>
-        <material name="rubber_tyre"/>
-      </visual>
-      <collision>
-        <origin xyz="0.0 0.0 0.0" rpy="0 0 0"/>
-        <geometry>
-          <mesh filename="$(find psd_vehicle_description)/meshes/stl/tyre.stl" scale="0.001 0.001 0.001"/>
-        </geometry>
-      </collision>
-    </link> -->
-    <!-- REAR -->
-    <link name="link_RL">
-      <inertial>
-        <origin xyz="0.0 0.0 0.0" rpy="0 0 0"/>
-        <mass value="0.270"/>
-        <inertia ixx="0.000189" iyy="0.000409" izz="0.000593" ixy="0.0" iyz="0.0" ixz="-0.0"/>
-      </inertial>
-      <visual>
-        <origin xyz="0.0 0.0 0.0" rpy="0 0 0"/>
-        <geometry>
-          <mesh filename="$(find psd_vehicle_description)/meshes/stl/suspension.stl" scale="0.001 0.001 0.001"/>
-        </geometry>
-        <material name="anodized_blue"/>
-      </visual>
-      <collision>
-        <origin xyz="0.0 0.0 0.0" rpy="0 0 0"/>
-        <geometry>
-          <mesh filename="$(find psd_vehicle_description)/meshes/stl/suspension.stl" scale="0.001 0.001 0.001"/>
-        </geometry>
-      </collision>
-    </link>
-    <link name="link_RR">
-      <inertial>
-        <origin xyz="0.0 0.0 0.0" rpy="0 0 0"/>
-        <mass value="0.270"/>
-        <inertia ixx="0.000189" iyy="0.000409" izz="0.000593" ixy="0.0" iyz="0.0" ixz="-0.0"/>
-      </inertial>
-      <visual>
-        <origin xyz="0.0 0.0 0.0" rpy="0 0 0"/>
-        <geometry>
-          <mesh filename="$(find psd_vehicle_description)/meshes/stl/suspension.stl" scale="0.001 0.001 0.001"/>
-        </geometry>
-        <material name="anodized_blue"/>
-      </visual>
-      <collision>
-        <origin xyz="0.0 0.0 0.0" rpy="0 0 0"/>
-        <geometry>
-          <mesh filename="$(find psd_vehicle_description)/meshes/stl/suspension.stl" scale="0.001 0.001 0.001"/>
-        </geometry>
-      </collision>
-    </link>
-    <link name="wheel_RL">
-      <inertial>
-        <origin xyz="0.0 0.0 0.0" rpy="0 0 0"/>
-        <mass value="2.80"/>
-        <inertia ixx="0.007152" iyy="0.005137" izz="0.005138" ixy="0.0" iyz="0.0" ixz="-0.0"/>
-      </inertial>
-      <visual>
-        <origin xyz="0.0 0.0 0.0" rpy="0 0 0"/>
-        <geometry>
-          <mesh filename="$(find psd_vehicle_description)/meshes/stl/wheel.stl" scale="0.001 0.001 0.001"/>
-        </geometry>
-        <material name="anodized_blue"/>
-      </visual>
-      <collision>
-        <origin xyz="0.0 0.0 0.0" rpy="0 0 0"/>
-        <geometry>
-          <!-- <mesh filename="$(find psd_vehicle_description)/meshes/stl/wheel.stl" scale="0.001 0.001 0.001"/> -->
-          <cylinder radius="${wheel_radius}" length="0.08"/>
-        </geometry>
-      </collision>
-    </link>
-    <link name="wheel_RR">
-      <inertial>
-        <origin xyz="0.0 0.0 0.0" rpy="0 0 0"/>
-        <mass value="2.80"/>
-        <inertia ixx="0.007152" iyy="0.005137" izz="0.005138" ixy="0.0" iyz="0.0" ixz="-0.0"/>
-      </inertial>
-      <visual>
-        <origin xyz="0.0 0.0 0.0" rpy="0 0 0"/>
-        <geometry>
-          <mesh filename="$(find psd_vehicle_description)/meshes/stl/wheel.stl" scale="0.001 0.001 0.001"/>
-        </geometry>
-        <material name="anodized_blue"/>
-      </visual>
-      <collision>
-        <origin xyz="0.0 0.0 0.0" rpy="0 0 0"/>
-        <geometry>
-          <!-- <mesh filename="$(find psd_vehicle_description)/meshes/stl/wheel.stl" scale="0.001 0.001 0.001"/> -->
-          <cylinder radius="${wheel_radius}" length="0.08"/>
-        </geometry>
-      </collision>
-    </link>
-    <!-- <link name="tyre_RL">
-      <inertial>
-        <origin xyz="0.0 0.0 0.0" rpy="0 0 0"/>
-        <mass value="4.40"/>
-        <inertia ixx="0.029818" iyy="0.017591" izz="0.017591" ixy="-0.0" iyz="0.0" ixz="0.0"/>
-      </inertial>
-      <visual>
-        <origin xyz="0.0 0.0 0.0" rpy="0 0 0"/>
-        <geometry>
-          <mesh filename="$(find psd_vehicle_description)/meshes/stl/tyre.stl" scale="0.001 0.001 0.001"/>
-        </geometry>
-        <material name="rubber_tyre"/>
-      </visual>
-      <collision>
-        <origin xyz="0.0 0.0 0.0" rpy="0 0 0"/>
-        <geometry>
-          <mesh filename="$(find psd_vehicle_description)/meshes/stl/tyre.stl" scale="0.001 0.001 0.001"/>
-        </geometry>
-      </collision>
-    </link>
-    <link name="tyre_RR">
-      <inertial>
-        <origin xyz="0.0 0.0 0.0" rpy="0 0 0"/>
-        <mass value="4.40"/>
-        <inertia ixx="0.029818" iyy="0.017591" izz="0.017591" ixy="-0.0" iyz="0.0" ixz="0.0"/>
-      </inertial>
-      <visual>
-        <origin xyz="0.0 0.0 0.0" rpy="0 0 0"/>
-        <geometry>
-          <mesh filename="$(find psd_vehicle_description)/meshes/stl/tyre.stl" scale="0.001 0.001 0.001"/>
-        </geometry>
-        <material name="rubber_tyre"/>
-      </visual>
-      <collision>
-        <origin xyz="0.0 0.0 0.0" rpy="0 0 0"/>
-        <geometry>
-          <mesh filename="$(find psd_vehicle_description)/meshes/stl/tyre.stl" scale="0.001 0.001 0.001"/>
-        </geometry>
-      </collision>
-    </link> -->
+        <origin xyz="-0.120217 -0.306869 -1.6e-05" rpy="0 0 0"/>
+        <geometry>
+          <mesh filename="$(find psd_vehicle_description)/meshes/collision/perno_FR_1.stl" scale="0.001 0.001 0.001"/>
+        </geometry>
+      </collision>
+    </link>
+    <link name="tyre_FR_1">
+      <inertial>
+        <origin xyz="0.03851831695141855 -0.017961168478880185 2.1642854608751476e-07" rpy="0 0 0"/>
+        <mass value="0.19445541180665865"/>
+        <inertia ixx="0.001191" iyy="0.000933" izz="0.000861" ixy="-0.000154" iyz="-0.0" ixz="0.0"/>
+      </inertial>
+      <visual>
+        <origin xyz="-0.122029 -0.306024 -1.6e-05" rpy="0 0 0"/>
+        <geometry>
+          <mesh filename="$(find psd_vehicle_description)/meshes/visual/tyre_FR_1.stl" scale="0.001 0.001 0.001"/>
+        </geometry>
+        <material name="anodized_blue"/>
+      </visual>
+      <collision>
+        <origin xyz="-0.122029 -0.306024 -1.6e-05" rpy="0 0 0"/>
+        <geometry>
+          <mesh filename="$(find psd_vehicle_description)/meshes/collision/tyre_FR_1.stl" scale="0.001 0.001 0.001"/>
+        </geometry>
+      </collision>
+    </link>
+    <link name="tyre_RR_1">
+      <inertial>
+        <origin xyz="0.04250016447333546 3.441685788030391e-07 2.16428546438244e-07" rpy="0 0 0"/>
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