Commit message: added custom_teleop_key and fixed typo on track.sdf

File: psd_ws/src/psd_vehicle_description/urdf/psd_vehicle_macro.ros2_control.xacro (robot description, xacro)
@@ -7,5 +7,5 @@
     <xacro:property name="PI" value="3.14159265359" />
     <xacro:property name="max_torque" value="100" />
-    <xacro:property name="max_steering_angle" value="${20 * PI / 180}" />
+    <xacro:property name="max_steering_angle" value="${30 * PI / 180}" />
     <ros2_control name="GazeboSimSystem" type="system">
       <hardware>

File: psd_ws/src/psd_vehicle_description/urdf/psd_vehicle_macro.urdf.xacro (robot description, xacro)
@@ -263,5 +263,5 @@
       <parent link="link_RR_1"/>
       <child link="tyre_RR_1"/>
-      <axis xyz="1.0 0.0 -0.0"/>
+      <axis xyz="-1.0 0.0 -0.0"/>
     </joint>
     <joint name="suspension_rl" type="fixed">
@@ -300,10 +300,10 @@
       rpy="0.0 0.0 0.0" />
     <!-- stereocamera -->
-    <!-- <xacro:include filename="$(find ros_components_description)/urdf/stereolabs_zed.urdf.xacro" ns="zed2" /> -->
+    <xacro:include filename="$(find ros_components_description)/urdf/intel_realsense_d435.urdf.xacro" ns="camera" />
     <!-- evaluate the macro and place the sensor on robot -->
-    <!-- <xacro:zed2.stereolabs_zed
+    <xacro:camera.intel_realsense_d435
       parent_link="chassis"
-      xyz="0.0 0.0 0.5"
-      rpy="0.0 0.0 0.0" /> -->
+      xyz="0.0 0.0 0.2"
+      rpy="0.0 0.0 ${3.1415/2}" />
   </xacro:macro>
 </robot>
