Commit message: added fake slam and fake perception

File: psd_ws/src/psd_vehicle_description/urdf/imu.xacro (robot description, xacro)
@@ -11,11 +11,4 @@
     <gazebo reference="imu_link">
         <sensor name="imu_sample" type="imu">
-            <!-- <plugin name="imu_controller" filename="libgz-imu-system.so">
-                <frame_name>imu_link</frame_name>
-                <ros>
-                    <remapping>~/out:=imu_broadcaster/imu</remapping>
-                </ros>
-                <initial_orientation_as_reference>false</initial_orientation_as_reference>
-            </plugin> -->
             <always_on>true</always_on>
             <update_rate>100</update_rate>

File: psd_ws/src/psd_vehicle_description/urdf/psd_vehicle.urdf.xacro (robot description, xacro)
@@ -3,9 +3,11 @@
   <xacro:include filename="$(find psd_vehicle_description)/urdf/psd_vehicle_macro.urdf.xacro"/>
   <xacro:include filename="$(find psd_vehicle_description)/urdf/psd_vehicle_macro.ros2_control.xacro"/>
+  <xacro:property name="PI" value="3.14159265359" />
+  <xacro:property name="rot90" value="${90 * PI / 180}" />
   <!-- Load robot's macro with parameters -->
   <link name="home" />
   <!-- set prefix if multiple robots are used -->
   <xacro:psd_vehicle parent="home" >
-    <origin xyz="0 0 0.095" rpy="0 0 0" />          <!-- position robot in the world -->
+    <origin xyz="0 0 0.095" rpy="0 0 -${rot90}" />          <!-- position robot in the world -->
   </xacro:psd_vehicle>
   <xacro:psd_vehicle_ros2_control

File: psd_ws/src/psd_vehicle_description/urdf/psd_vehicle_macro.urdf.xacro (robot description, xacro)
@@ -237,4 +237,11 @@
       xyz="0.0 0.0 0.2"
       rpy="0.0 0.0 ${rot90}" />
+    <!-- position/odom -->
+    <link name="base_footprint"/>
+    <joint name="footprint_joint" type="fixed">
+      <parent link="chassis"/>
+      <child link="base_footprint"/>
+      <origin xyz="0.0 0.0 0.0" rpy="0 0 0"/>
+    </joint>
   </xacro:macro>
 </robot>
