Commit message: starting ROS2 Jazzy migration and Gazebo gz Harmonic

File: psd_ws/install/psd_vehicle_description/share/psd_vehicle_description/urdf/components/camera_mount.urdf.xacro (robot description, xacro)
@@ -1 +1,85 @@
-/home/psd/psd_ws/src/psd_vehicle_description/urdf/components/camera_mount.urdf.xacro
+<?xml version="1.0"?>
+<robot xmlns:xacro="http://www.ros.org/wiki/xacro">
+  <xacro:macro name="camera_mount"
+    params="parent_link xyz rpy
+                       tf_prefix:=None
+                       camera_mount_angle_1:=0.0
+                       camera_mount_angle_2:=0.0">
+    <xacro:if value="${tf_prefix == 'None'}">
+      <xacro:property name="tf_prefix_ext" value="" />
+    </xacro:if>
+    <xacro:unless value="${tf_prefix == 'None'}">
+      <xacro:property name="tf_prefix_ext" value="${tf_prefix}_" />
+    </xacro:unless>
+    <joint name="${parent_link.rstrip('_link')}_to_${tf_prefix_ext}camera_mount_bot_joint"
+      type="fixed">
+      <origin xyz="${xyz}" rpy="${rpy}" />
+      <parent link="${parent_link}" />
+      <child link="${tf_prefix_ext}camera_mount_bot_link" />
+    </joint>
+    <link name="${tf_prefix_ext}camera_mount_bot_link">
+      <visual>
+        <geometry>
+          <mesh filename="file://$(find psd_vehicle_description)/meshes/components/camera_mount_bot.dae"
+      scale="1 1 1" />
+        </geometry>
+        <origin xyz="0.0 0.0 0.0" rpy="0.0 0.0 0.0" />
+      </visual>
+      <collision>
+        <geometry>
+          <box size="0.0275 0.0275 0.023" />
+        </geometry>
+        <origin xyz="0.0 0.0 0.0115" rpy="0.0 0.0 0.0" />
+      </collision>
+    </link>
+    <joint name="${tf_prefix_ext}camera_mount_bot_to_${tf_prefix_ext}camera_mount_mid_joint"
+      type="fixed">
+      <origin xyz="0.0 0.0 0.016" rpy="0.0 ${camera_mount_angle_1} 0.0" />
+      <parent link="${tf_prefix_ext}camera_mount_bot_link" />
+      <child link="${tf_prefix_ext}camera_mount_mid_link" />
+    </joint>
+    <link name="${tf_prefix_ext}camera_mount_mid_link">
+      <visual>
+        <geometry>
+          <mesh filename="file://$(find psd_vehicle_description)/meshes/components/camera_mount_mid.dae"
+      scale="1 1 1" />
+        </geometry>
+        <origin xyz="0.0 0.0 0.0" rpy="0.0 0.0 0.0" />
+      </visual>
+      <collision>
+        <geometry>
+          <box size="0.015 0.017 0.101" />
+        </geometry>
+        <origin xyz="0.0 0.0 0.0425" rpy="0.0 0.0 0.0" />
+      </collision>
+    </link>
+    <joint name="${tf_prefix_ext}camera_mount_mid_to_${tf_prefix_ext}camera_mount_top_joint"
+      type="fixed">
+      <origin xyz="0.0 0.0 0.086" rpy="0.0 ${camera_mount_angle_2} 0.0" />
+      <parent link="${tf_prefix_ext}camera_mount_mid_link" />
+      <child link="${tf_prefix_ext}camera_mount_top_link" />
+    </joint>
+    <link name="${tf_prefix_ext}camera_mount_top_link">
+      <visual>
+        <geometry>
+          <mesh filename="file://$(find psd_vehicle_description)/meshes/components/camera_mount_top.dae"
+      scale="1 1 1" />
+        </geometry>
+        <origin xyz="0.0 0.0 0.0" rpy="0.0 0.0 0.0" />
+      </visual>
+      <collision>
+        <geometry>
+          <box size="0.023 0.023 0.025" />
+        </geometry>
+        <origin xyz="0.0 -0.00232 0.0065" rpy="0.0 0.0 0.0" />
+      </collision>
+    </link>
+    <joint name="${tf_prefix_ext}camera_mount_top_to_${tf_prefix_ext}camera_mount_joint"
+      type="fixed">
+      <origin xyz="0.0 -0.00232 0.019" rpy="0.0 0.0 0.0" />
+      <parent link="${tf_prefix_ext}camera_mount_top_link" />
+      <child link="${tf_prefix_ext}camera_mount_link" />
+    </joint>
+    <link name="${tf_prefix_ext}camera_mount_link" />
+  </xacro:macro>
+</robot>

File: psd_ws/install/psd_vehicle_description/share/psd_vehicle_description/urdf/materials.xacro (robot description, xacro)
@@ -1 +1,52 @@
-/home/psd/psd_ws/src/psd_vehicle_description/urdf/materials.xacro
+<?xml version="1.0" encoding="UTF-8"?>
+<robot name="psd_vehicle" xmlns:xacro="http://www.ros.org/wiki/xacro" >
+  <material name="silver">
+    <color rgba="0.70 0.70 0.70 1.000"/>
+    <lighting>1</lighting> <!-- Enable lighting effects -->
+    <ambient>0.1 0.1 0.1 1.0</ambient> <!-- Ambient light color -->
+    <diffuse>0.6 0.6 0.6 1.0</diffuse> <!-- Diffuse reflection color -->
+    <specular>0.3 0.3 0.3 1.0</specular> <!-- Specular reflection color -->
+    <emissive>0.0 0.0 0.0 1.0</emissive> <!-- Emissive color -->
+    <transparency>0.0</transparency> <!-- Transparency (0.0 for opaque) -->
+  </material>
+  <material name="anodized_red">
+    <color rgba="1.0 0.0 0.0 1.000"/>
+    <lighting>1</lighting> <!-- Enable lighting effects -->
+    <ambient>0.1 0.1 0.1 1.0</ambient> <!-- Ambient light color -->
+    <diffuse>0.6 0.6 0.6 1.0</diffuse> <!-- Diffuse reflection color -->
+    <specular>0.3 0.3 0.3 1.0</specular> <!-- Specular reflection color -->
+    <emissive>0.0 0.0 0.0 1.0</emissive> <!-- Emissive color -->
+    <transparency>0.0</transparency> <!-- Transparency (0.0 for opaque) -->
+  </material>
+  <material name="anodized_blue">
+    <color rgba="0.0 0.5 1.0 1.0"/> <!-- Blue color with full opacity -->
+    <lighting>1</lighting> <!-- Enable lighting effects -->
+    <ambient>0.1 0.1 0.1 1.0</ambient> <!-- Ambient light color -->
+    <diffuse>0.6 0.6 0.6 1.0</diffuse> <!-- Diffuse reflection color -->
+    <specular>0.3 0.3 0.3 1.0</specular> <!-- Specular reflection color -->
+    <emissive>0.0 0.0 0.0 1.0</emissive> <!-- Emissive color -->
+    <transparency>0.0</transparency> <!-- Transparency (0.0 for opaque) -->
+  </material>
+  <material name="rubber_tyre">
+    <color rgba="0.0 0.0 0.0 1.000"/>
+    <lighting>1</lighting> <!-- Enable lighting effects -->
+    <ambient>0.1 0.1 0.1 1.0</ambient> <!-- Ambient light color -->
+    <diffuse>0.6 0.6 0.6 1.0</diffuse> <!-- Diffuse reflection color -->
+    <specular>0.3 0.3 0.3 1.0</specular> <!-- Specular reflection color -->
+    <emissive>0.0 0.0 0.0 1.0</emissive> <!-- Emissive color -->
+    <transparency>0.0</transparency> <!-- Transparency (0.0 for opaque) -->
+    <friction>
+      <ode>
+        <mu>0.8</mu> <!-- Friction coefficient -->
+        <mu2>0.8</mu2> <!-- Friction coefficient -->
+      </ode>
+    </friction>
+    <elasticity>
+      <ode>
+        <epsilon>0.8</epsilon> <!-- Coefficient of restitution (elasticity) -->
+        <kp>100000000.0</kp> <!-- Contact stiffness -->
+        <kd>10.0</kd> <!-- Contact damping -->
+      </ode>
+    </elasticity>
+  </material>
+</robot>

File: psd_ws/install/psd_vehicle_description/share/psd_vehicle_description/urdf/psd_vehicle.urdf.xacro (robot description, xacro)
@@ -1 +1,18 @@
-/home/psd/psd_ws/src/psd_vehicle_description/urdf/psd_vehicle.urdf.xacro
+<?xml version="1.0" encoding="UTF-8"?>
+<robot xmlns:xacro="http://wiki.ros.org/xacro" name="psd_vehicle">
+  <!-- Use this if parameters are set from the launch file, otherwise delete -->
+  <xacro:arg name="prefix" default="" />
+  <xacro:arg name="simulation_controllers" default="" />
+  <xacro:include filename="$(find psd_vehicle_description)/urdf/psd_vehicle_macro.urdf.xacro"/>
+  <xacro:include filename="$(find psd_vehicle_description)/urdf/psd_vehicle_macro.ros2_control.xacro"/>
+  <!-- Load robot's macro with parameters -->
+  <link name="leo" />
+  <!-- set prefix if multiple robots are used -->
+  <xacro:psd_vehicle prefix="$(arg prefix)" parent="leo" >
+    <origin xyz="0 0 0.095" rpy="0 0 0" />          <!-- position robot in the world -->
+  </xacro:psd_vehicle>
+  <xacro:psd_vehicle_ros2_control
+    name="psd_vehicle"
+    prefix="$(arg prefix)"
+  />
+</robot>

File: psd_ws/install/psd_vehicle_description/share/psd_vehicle_description/urdf/psd_vehicle_macro.ros2_control.xacro (robot description, xacro)
@@ -1 +1,68 @@
-/home/psd/psd_ws/src/psd_vehicle_description/urdf/psd_vehicle_macro.ros2_control.xacro
+<?xml version='1.0'?>
+<robot xmlns:xacro="http://wiki.ros.org/xacro">
+  <xacro:macro name="psd_vehicle_ros2_control" params="
+                name
+                prefix
+                use_mock_hardware:=^|false
+                mock_sensor_commands:=^|false
+                sim_gazebo:=^|false"
+                >
+    <ros2_control name="${name}" type="system">
+      <hardware>
+        <xacro:if value="${use_mock_hardware}">
+          <plugin>mock_components/GenericSystem</plugin>
+          <param name="mock_sensor_commands">${mock_sensor_commands}</param>
+        </xacro:if>
+        <xacro:if value="${sim_gazebo}">
+          <plugin>ign_ros2_control/IgnitionSystem</plugin>
+        </xacro:if>
+      </hardware>
+      <joint name="${prefix}steering_fl">
+        <command_interface name="position"/>
+        <state_interface name="position"/>
+      </joint>
+      <joint name="${prefix}steering_fr">
+        <command_interface name="position"/>
+        <state_interface name="position"/>
+      </joint>
+      <joint name="${prefix}drive_rl">
+        <command_interface name="effort"/>
+        <state_interface name="position"/>
+        <state_interface name="velocity"/>
+      </joint>
+      <joint name="${prefix}drive_rr">
+        <command_interface name="effort"/>
+        <state_interface name="position"/>
+        <state_interface name="velocity"/>
+      </joint>
+      <joint name="${prefix}drive_fl">
+        <command_interface name="effort"/>
+        <state_interface name="position"/>
+        <state_interface name="velocity"/>
+      </joint>
+      <joint name="${prefix}drive_fr">
+        <command_interface name="effort"/>
+        <state_interface name="position"/>
+        <state_interface name="velocity"/>
+      </joint>
+      <sensor name="tcp_fts_sensor1">
+        <state_interface name="fx"/>
+        <state_interface name="fy"/>
+        <state_interface name="fz"/>
+        <state_interface name="tx"/>
+        <state_interface name="ty"/>
+        <state_interface name="tz"/>
+        <param name="frame_id">tyre_RL_1</param>
+      </sensor>
+      <sensor name="tcp_fts_sensor2">
+        <state_interface name="fx"/>
+        <state_interface name="fy"/>
+        <state_interface name="fz"/>
+        <state_interface name="tx"/>
+        <state_interface name="ty"/>
+        <state_interface name="tz"/>
+        <param name="frame_id">tyre_RR_1</param>
+      </sensor>
+    </ros2_control>
+  </xacro:macro>
+</robot>
