Commit message: starting ROS2 Jazzy migration and Gazebo gz Harmonic

File: psd_ws/install/psd_vehicle_description/share/psd_vehicle_description/urdf/psd_vehicle_macro.urdf.xacro (robot description, xacro)
@@ -1 +1,297 @@
-/home/psd/psd_ws/src/psd_vehicle_description/urdf/psd_vehicle_macro.urdf.xacro
+<?xml version="1.0" ?>
+<robot name="psd_vehicle" xmlns:xacro="http://www.ros.org/wiki/xacro">
+  <!-- include materials -->
+  <xacro:include filename="$(find psd_vehicle_description)/urdf/materials.xacro" />
+  <!-- start vehicle description -->
+  <xacro:macro name="psd_vehicle" params="prefix parent *origin">
+    <!-- LINKS -->
+    <!-- Chassis START-->
+    <link name="${prefix}chassis">
+      <inertial>
+        <origin xyz="-0.055282024534886974 0.006459558608433099 1.621642854614675e-05" rpy="0 0 0"/>
+        <mass value="7.077984465449566"/>
+        <inertia ixx="0.233109" iyy="0.053798" izz="0.264742" ixy="-0.0" iyz="-0.0" ixz="-0.0"/>
+      </inertial>
+      <visual>
+        <origin xyz="0 0 0" rpy="0 0 0"/>
+        <geometry>
+          <mesh filename="$(find psd_vehicle_description)/meshes/visual/base_link.stl" scale="0.001 0.001 0.001"/>
+        </geometry>
+        <material name="anodized_red"/>
+      </visual>
+      <collision>
+        <origin xyz="0 0 0" rpy="0 0 0"/>
+        <geometry>
+          <mesh filename="$(find psd_vehicle_description)/meshes/collision/base_link.stl" scale="0.001 0.001 0.001"/>
+        </geometry>
+      </collision>
+    </link>
+    <joint name="${prefix}world_joint" type="fixed">
+      <xacro:insert_block name="origin" />
+      <parent link="${parent}" />
+      <child link="${prefix}chassis" />
+    </joint>
+    <link name="${prefix}perno_FL_1">
+      <inertial>
+        <origin xyz="-0.000906687358749575 0.00042296243032097225 2.1642838935455414e-07" rpy="0 0 0"/>
+        <mass value="0.00011097676048806171"/>
+        <inertia ixx="0.0" iyy="0.0" izz="0.0" ixy="-0.0" iyz="0.0" ixz="-0.0"/>
+      </inertial>
+      <visual>
+        <origin xyz="0.230783 -0.306869 -1.6e-05" rpy="0 0 0"/>
+        <geometry>
+          <mesh filename="$(find psd_vehicle_description)/meshes/visual/perno_FL_1.stl" scale="0.001 0.001 0.001"/>
+        </geometry>
+        <material name="silver"/>
+      </visual>
+      <collision>
+        <origin xyz="0.230783 -0.306869 -1.6e-05" rpy="0 0 0"/>
+        <geometry>
+          <mesh filename="$(find psd_vehicle_description)/meshes/collision/perno_FL_1.stl" scale="0.001 0.001 0.001"/>
+        </geometry>
+      </collision>
+    </link>
+    <link name="${prefix}tyre_FL_1">
+      <inertial>
+        <origin xyz="-0.03851807609484373 0.017960856816041648 2.1642854673904234e-07" rpy="0 0 0"/>
+        <mass value="0.1944554118066591"/>
+        <inertia ixx="0.001191" iyy="0.000933" izz="0.000861" ixy="-0.000154" iyz="0.0" ixz="0.0"/>
+      </inertial>
+      <visual>
+        <origin xyz="0.232596 -0.307715 -1.6e-05" rpy="0 0 0"/>
+        <geometry>
+          <mesh filename="$(find psd_vehicle_description)/meshes/visual/tyre_FL_1.stl" scale="0.001 0.001 0.001"/>
+        </geometry>
+        <material name="rubber_tyre"/>
+      </visual>
+      <collision>
+        <origin xyz="0.232596 -0.307715 -1.6e-05" rpy="0 0 0"/>
+        <geometry>
+          <mesh filename="$(find psd_vehicle_description)/meshes/collision/tyre_FL_1.stl" scale="0.001 0.001 0.001"/>
+        </geometry>
+      </collision>
+    </link>z
+    <link name="${prefix}perno_FR_1">
+      <inertial>
+        <origin xyz="0.000905928215323884 -0.0004222740931605351 2.1642839664261197e-07" rpy="0 0 0"/>
+        <mass value="0.0001109767604880609"/>
+        <inertia ixx="0.0" iyy="0.0" izz="0.0" ixy="-0.0" iyz="-0.0" ixz="0.0"/>
+      </inertial>
+      <visual>
+        <origin xyz="-0.120217 -0.306869 -1.6e-05" rpy="0 0 0"/>
+        <geometry>
+          <mesh filename="$(find psd_vehicle_description)/meshes/visual/perno_FR_1.stl" scale="0.001 0.001 0.001"/>
+        </geometry>
+        <material name="silver"/>
+      </visual>
+      <collision>
+        <origin xyz="-0.120217 -0.306869 -1.6e-05" rpy="0 0 0"/>
+        <geometry>
+          <mesh filename="$(find psd_vehicle_description)/meshes/collision/perno_FR_1.stl" scale="0.001 0.001 0.001"/>
+        </geometry>
+      </collision>
+    </link>
+    <link name="${prefix}tyre_FR_1">
+      <inertial>
+        <origin xyz="0.03851831695141855 -0.017961168478880185 2.1642854608751476e-07" rpy="0 0 0"/>
+        <mass value="0.19445541180665865"/>
+        <inertia ixx="0.001191" iyy="0.000933" izz="0.000861" ixy="-0.000154" iyz="-0.0" ixz="0.0"/>
+      </inertial>
+      <visual>
+        <origin xyz="-0.122029 -0.306024 -1.6e-05" rpy="0 0 0"/>
+        <geometry>
+          <mesh filename="$(find psd_vehicle_description)/meshes/visual/tyre_FR_1.stl" scale="0.001 0.001 0.001"/>
+        </geometry>
+        <material name="rubber_tyre"/>
+      </visual>
+      <collision>
+        <origin xyz="-0.122029 -0.306024 -1.6e-05" rpy="0 0 0"/>
+        <geometry>
+          <mesh filename="$(find psd_vehicle_description)/meshes/collision/tyre_FR_1.stl" scale="0.001 0.001 0.001"/>
+        </geometry>
+      </collision>
+    </link>
+    <link name="${prefix}tyre_RR_1">
+      <inertial>
+        <origin xyz="0.04250016447333546 3.441685788030391e-07 2.16428546438244e-07" rpy="0 0 0"/>
+        <mass value="0.19445541180665948"/>
+        <inertia ixx="0.001262" iyy="0.000861" izz="0.000861" ixy="-0.0" iyz="-0.0" ixz="0.0"/>
+      </inertial>
+      <visual>
+        <origin xyz="-0.119284 0.293131 -1.6e-05" rpy="0 0 0"/>
+        <geometry>
+          <mesh filename="$(find psd_vehicle_description)/meshes/visual/tyre_RR_1.stl" scale="0.001 0.001 0.001"/>
+        </geometry>
+        <material name="rubber_tyre"/>
+      </visual>
+      <collision>
+        <origin xyz="-0.119284 0.293131 -1.6e-05" rpy="0 0 0"/>
+        <geometry>
+          <mesh filename="$(find psd_vehicle_description)/meshes/collision/tyre_RR_1.stl" scale="0.001 0.001 0.001"/>
+        </geometry>
+      </collision>
+    </link>
+    <link name="${prefix}link_RL_1">
+      <inertial>
+        <origin xyz="-0.047944553368047954 3.441685789140614e-07 2.1642854618965338e-07" rpy="0 0 0"/>
+        <mass value="0.09195911794645473"/>
+        <inertia ixx="6.5e-05" iyy="0.000142" izz="0.000206" ixy="-0.0" iyz="0.0" ixz="0.0"/>
+      </inertial>
+      <visual>
+        <origin xyz="0.095283 0.293131 -1.6e-05" rpy="0 0 0"/>
+        <geometry>
+          <mesh filename="$(find psd_vehicle_description)/meshes/visual/link_RL_1.stl" scale="0.001 0.001 0.001"/>
+        </geometry>
+        <material name="anodized_blue"/>
+      </visual>
+      <collision>
+        <origin xyz="0.095283 0.293131 -1.6e-05" rpy="0 0 0"/>
+        <geometry>
+          <mesh filename="$(find psd_vehicle_description)/meshes/collision/link_RL_1.stl" scale="0.001 0.001 0.001"/>
+        </geometry>
+      </collision>
+    </link>
+    <link name="${prefix}link_RR_1">
+      <inertial>
+        <origin xyz="0.04794379422462264 3.441685790250837e-07 2.1642854618632285e-07" rpy="0 0 0"/>
+        <mass value="0.09195911794645475"/>
+        <inertia ixx="6.5e-05" iyy="0.000142" izz="0.000206" ixy="0.0" iyz="-0.0" ixz="0.0"/>
+      </inertial>
+      <visual>
+        <origin xyz="0.015283 0.293131 -1.6e-05" rpy="0 0 0"/>
+        <geometry>
+          <mesh filename="$(find psd_vehicle_description)/meshes/visual/link_RR_1.stl" scale="0.001 0.001 0.001"/>
+        </geometry>
+        <material name="anodized_blue"/>
+      </visual>
+      <collision>
+        <origin xyz="0.015283 0.293131 -1.6e-05" rpy="0 0 0"/>
+        <geometry>
+          <mesh filename="$(find psd_vehicle_description)/meshes/collision/link_RR_1.stl" scale="0.001 0.001 0.001"/>
+        </geometry>
+      </collision>
+    </link>
+    <link name="${prefix}tyre_RL_1">
+      <inertial>
+        <origin xyz="-0.04249992361676111 3.4416857908059484e-07 2.1642854653184114e-07" rpy="0 0 0"/>
+        <mass value="0.19445541180665912"/>
+        <inertia ixx="0.001262" iyy="0.000861" izz="0.000861" ixy="0.0" iyz="0.0" ixz="0.0"/>
+      </inertial>
+      <visual>
+        <origin xyz="0.229851 0.293131 -1.6e-05" rpy="0 0 0"/>
+        <geometry>
+          <mesh filename="$(find psd_vehicle_description)/meshes/visual/tyre_RL_1.stl" scale="0.001 0.001 0.001"/>
+        </geometry>
+        <material name="rubber_tyre"/>
+      </visual>
+      <collision>
+        <origin xyz="0.229851 0.293131 -1.6e-05" rpy="0 0 0"/>
+        <geometry>
+          <mesh filename="$(find psd_vehicle_description)/meshes/collision/tyre_RL_1.stl" scale="0.001 0.001 0.001"/>
+        </geometry>
+      </collision>
+    </link>
+    <link name="${prefix}link_FL_1">
+      <inertial>
+        <origin xyz="-0.04795315128569644 3.441685794691729e-07 2.1642854620519813e-07" rpy="0 0 0"/>
+        <mass value="0.09196821373647668"/>
+        <inertia ixx="6.5e-05" iyy="0.000142" izz="0.000206" ixy="0.0" iyz="0.0" ixz="-0.0"/>
+      </inertial>
+      <visual>
+        <origin xyz="0.095283 -0.306869 -1.6e-05" rpy="0 0 0"/>
+        <geometry>
+          <mesh filename="$(find psd_vehicle_description)/meshes/visual/link_FL_1.stl" scale="0.001 0.001 0.001"/>
+        </geometry>
+        <material name="anodized_blue"/>
+      </visual>
+      <collision>
+        <origin xyz="0.095283 -0.306869 -1.6e-05" rpy="0 0 0"/>
+        <geometry>
+          <mesh filename="$(find psd_vehicle_description)/meshes/collision/link_FL_1.stl" scale="0.001 0.001 0.001"/>
+        </geometry>
+      </collision>
+    </link>
+    <link name="${prefix}link_FR_1">
+      <inertial>
+        <origin xyz="0.04795239214227047 3.441685796912175e-07 2.164285462018676e-07" rpy="0 0 0"/>
+        <mass value="0.09196821373647673"/>
+        <inertia ixx="6.5e-05" iyy="0.000142" izz="0.000206" ixy="-0.0" iyz="0.0" ixz="0.0"/>
+      </inertial>
+      <visual>
+        <origin xyz="0.015283 -0.306869 -1.6e-05" rpy="0 0 0"/>
+        <geometry>
+          <mesh filename="$(find psd_vehicle_description)/meshes/visual/link_FR_1.stl" scale="0.001 0.001 0.001"/>
+        </geometry>
+        <material name="anodized_blue"/>
+      </visual>
+      <collision>
+        <origin xyz="0.015283 -0.306869 -1.6e-05" rpy="0 0 0"/>
+        <geometry>
+          <mesh filename="$(find psd_vehicle_description)/meshes/collision/link_FR_1.stl" scale="0.001 0.001 0.001"/>
+        </geometry>
+      </collision>
+    </link>
+    <!-- JOINTS -->
+    <joint name="${prefix}steering_fl" type="revolute">
+      <origin xyz="-0.1355 0.0 0.0" rpy="0 0 0"/>
+      <parent link="${prefix}link_FL_1"/>
+      <child link="${prefix}perno_FL_1"/>
+      <axis xyz="0.0 -0.0 1.0"/>
+      <limit upper="0.523599" lower="-0.523599" effort="100" velocity="100"/>
+      <mimic joint="${prefix}steering_fr" multiplier="1.0" offset="0.0"/>
+    </joint>
+    <joint name="${prefix}drive_fl" type="continuous">
+      <origin xyz="-0.001813 0.000846 0.0" rpy="0 0 0"/>
+      <parent link="${prefix}perno_FL_1"/>
+      <child link="${prefix}tyre_FL_1"/>
+      <axis xyz="-0.906308 0.422618 0.0"/>
+      <mimic joint="${prefix}drive_rl" multiplier="1.0" offset="0.0"/>
+    </joint>
+    <joint name="${prefix}steering_fr" type="revolute">
+      <origin xyz="0.1355 0.0 0.0" rpy="0 0 0"/>
+      <parent link="${prefix}link_FR_1"/>
+      <child link="${prefix}perno_FR_1"/>
+      <axis xyz="0.0 -0.0 1.0"/>
+      <limit upper="0.523599" lower="-0.523599" effort="100" velocity="100"/>
+    </joint>
+    <joint name="${prefix}drive_fr" type="continuous">
+      <origin xyz="0.001812 -0.000845 0.0" rpy="0 0 0"/>
+      <parent link="${prefix}perno_FR_1"/>
+      <child link="${prefix}tyre_FR_1"/>
+      <axis xyz="0.906308 -0.422618 -0.0"/>
+      <mimic joint="${prefix}drive_rr" multiplier="1.0" offset="0.0"/>
+    </joint>
+    <joint name="${prefix}drive_rr" type="continuous">
+      <origin xyz="0.134567 0.0 0.0" rpy="0 0 0"/>
+      <parent link="${prefix}link_RR_1"/>
+      <child link="${prefix}tyre_RR_1"/>
+      <axis xyz="1.0 0.0 -0.0"/>
+    </joint>
+    <joint name="${prefix}suspension_rl" type="fixed">
+      <origin xyz="-0.095283 -0.293131 1.6e-05" rpy="0 0 0"/>
+      <parent link="${prefix}chassis"/>
+      <child link="${prefix}link_RL_1"/>
+    </joint>
+    <joint name="${prefix}suspension_rr" type="fixed">
+      <origin xyz="-0.015283 -0.293131 1.6e-05" rpy="0 0 0"/>
+      <parent link="${prefix}chassis"/>
+      <child link="${prefix}link_RR_1"/>
+    </joint>
+    <joint name="${prefix}drive_rl" type="continuous">
+      <origin xyz="-0.134568 0.0 0.0" rpy="0 0 0"/>
+      <parent link="${prefix}link_RL_1"/>
+      <child link="${prefix}tyre_RL_1"/>
+      <axis xyz="-1.0 -0.0 0.0"/>
+    </joint>
+    <joint name="${prefix}suspension_fl" type="fixed">
+      <origin xyz="-0.095283 0.306869 1.6e-05" rpy="0 0 0"/>
+      <parent link="${prefix}chassis"/>
+      <child link="${prefix}link_FL_1"/>
+    </joint>
+    <joint name="${prefix}suspension_fr" type="fixed">
+      <origin xyz="-0.015283 0.306869 1.6e-05" rpy="0 0 0"/>
+      <parent link="${prefix}chassis"/>
+      <child link="${prefix}link_FR_1"/>
+    </joint>
+  </xacro:macro>
+</robot>

File: psd_ws/src/psd_vehicle_description/urdf/psd_vehicle.urdf.xacro (robot description, xacro)
@@ -7,7 +7,7 @@
   <xacro:include filename="$(find psd_vehicle_description)/urdf/psd_vehicle_macro.ros2_control.xacro"/>
   <!-- Load robot's macro with parameters -->
-  <link name="world" />
+  <link name="leo" />
   <!-- set prefix if multiple robots are used -->
-  <xacro:psd_vehicle prefix="$(arg prefix)" parent="world" >
+  <xacro:psd_vehicle prefix="$(arg prefix)" parent="leo" >
     <origin xyz="0 0 0.095" rpy="0 0 0" />          <!-- position robot in the world -->
   </xacro:psd_vehicle>

File: psd_ws/src/psd_vehicle_description/urdf/psd_vehicle_macro.ros2_control.xacro (robot description, xacro)
@@ -3,7 +3,19 @@
   <xacro:macro name="psd_vehicle_ros2_control" params="
                 name
-                prefix"
+                prefix
+                use_mock_hardware:=^|false
+                mock_sensor_commands:=^|false
+                sim_gazebo:=^|false"
                 >
     <ros2_control name="${name}" type="system">
+      <hardware>
+        <xacro:if value="${use_mock_hardware}">
+          <plugin>mock_components/GenericSystem</plugin>
+          <param name="mock_sensor_commands">${mock_sensor_commands}</param>
+        </xacro:if>
+        <xacro:if value="${sim_gazebo}">
+          <plugin>ign_ros2_control/IgnitionSystem</plugin>
+        </xacro:if>
+      </hardware>
       <joint name="${prefix}steering_fl">
         <command_interface name="position"/>

File: psd_ws/src/psd_vehicle_description/urdf/psd_vehicle_macro.urdf.xacro (robot description, xacro)
@@ -6,37 +6,30 @@
   <xacro:macro name="psd_vehicle" params="prefix parent *origin">
     <!-- LINKS -->
-    <!-- base link -->
-    <link name="${prefix}base_link" />
+    <!-- Chassis START-->
+    <link name="${prefix}chassis">
+      <inertial>
+        <origin xyz="-0.055282024534886974 0.006459558608433099 1.621642854614675e-05" rpy="0 0 0"/>
+        <mass value="7.077984465449566"/>
+        <inertia ixx="0.233109" iyy="0.053798" izz="0.264742" ixy="-0.0" iyz="-0.0" ixz="-0.0"/>
+      </inertial>
+      <visual>
+        <origin xyz="0 0 0" rpy="0 0 0"/>
+        <geometry>
+          <mesh filename="$(find psd_vehicle_description)/meshes/visual/base_link.stl" scale="0.001 0.001 0.001"/>
+        </geometry>
+        <material name="anodized_red"/>
+      </visual>
+      <collision>
+        <origin xyz="0 0 0" rpy="0 0 0"/>
+        <geometry>
+          <mesh filename="$(find psd_vehicle_description)/meshes/collision/base_link.stl" scale="0.001 0.001 0.001"/>
+        </geometry>
+      </collision>
+    </link>
     <joint name="${prefix}world_joint" type="fixed">
       <xacro:insert_block name="origin" />
       <parent link="${parent}" />
-      <child link="${prefix}base_link" />
-    </joint>
-    <!-- Chassis START-->
-    <joint name="${prefix}base_joint" type="fixed">
-      <origin xyz="0.0 0.0 0.0" rpy="0.0 0.0 0.0" />
-      <parent link="${prefix}base_link"/>
-      <child link="${prefix}chassis"/>
-    </joint>
-    <link name="${prefix}chassis">
-      <inertial>
-        <origin xyz="-0.055282024534886974 0.006459558608433099 1.621642854614675e-05" rpy="0 0 0"/>
-        <mass value="7.077984465449566"/>
-        <inertia ixx="0.233109" iyy="0.053798" izz="0.264742" ixy="-0.0" iyz="-0.0" ixz="-0.0"/>
-      </inertial>
-      <visual>
-        <origin xyz="0 0 0" rpy="0 0 0"/>
-        <geometry>
-          <mesh filename="$(find psd_vehicle_description)/meshes/visual/base_link.stl" scale="0.001 0.001 0.001"/>
-        </geometry>
-        <material name="anodized_red"/>
-      </visual>
-      <collision>
-        <origin xyz="0 0 0" rpy="0 0 0"/>
-        <geometry>
-          <mesh filename="$(find psd_vehicle_description)/meshes/collision/base_link.stl" scale="0.001 0.001 0.001"/>
-        </geometry>
-      </collision>
-    </link>
+      <child link="${prefix}chassis" />
+    </joint>
     <link name="${prefix}perno_FL_1">
       <inertial>
@@ -301,156 +294,4 @@
       <child link="${prefix}link_FR_1"/>
     </joint>
-    <!-- ############## SENSORS ############## -->
-    <link name="${prefix}imu_link">
-      <visual>
-        <geometry>
-          <box size="0.1 0.1 0.1"/>
-        </geometry>
-      </visual>
-      <collision>
-        <geometry>
-          <box size="0.1 0.1 0.1"/>
-        </geometry>
-      </collision>
-    </link>
-    <joint name="${prefix}imu_joint" type="fixed">
-      <parent link="${prefix}chassis"/>
-      <child link="${prefix}imu_link"/>
-      <origin xyz="0 0 0.01"/>
-    </joint>
-    <gazebo reference="${prefix}imu_link">
-      <sensor name="imu_sensor" type="imu">
-      <plugin filename="libgazebo_ros_imu_sensor.so" name="imu_plugin">
-          <ros>
-            <namespace>/demo</namespace>
-            <remapping>~/out:=imu</remapping>
-          </ros>
-          <initial_orientation_as_reference>false</initial_orientation_as_reference>
-        </plugin>
-        <always_on>true</always_on>
-        <update_rate>100</update_rate>
-        <visualize>true</visualize>
-        <imu>
-          <angular_velocity>
-            <x>
-              <noise type="gaussian">
-                <mean>0.0</mean>
-                <stddev>2e-4</stddev>
-                <bias_mean>0.0000075</bias_mean>
-                <bias_stddev>0.0000008</bias_stddev>
-              </noise>
-            </x>
-            <y>
-              <noise type="gaussian">
-                <mean>0.0</mean>
-                <stddev>2e-4</stddev>
-                <bias_mean>0.0000075</bias_mean>
-                <bias_stddev>0.0000008</bias_stddev>
-              </noise>
-            </y>
-            <z>
-              <noise type="gaussian">
-                <mean>0.0</mean>
-                <stddev>2e-4</stddev>
-                <bias_mean>0.0000075</bias_mean>
-                <bias_stddev>0.0000008</bias_stddev>
-              </noise>
-            </z>
-          </angular_velocity>
-          <linear_acceleration>
-            <x>
-              <noise type="gaussian">
-                <mean>0.0</mean>
-                <stddev>1.7e-2</stddev>
-                <bias_mean>0.1</bias_mean>
-                <bias_stddev>0.001</bias_stddev>
-              </noise>
-            </x>
-            <y>
-              <noise type="gaussian">
-                <mean>0.0</mean>
-                <stddev>1.7e-2</stddev>
-                <bias_mean>0.1</bias_mean>
-                <bias_stddev>0.001</bias_stddev>
-              </noise>
-            </y>
-            <z>
-              <noise type="gaussian">
-                <mean>0.0</mean>
-                <stddev>1.7e-2</stddev>
-                <bias_mean>0.1</bias_mean>
-                <bias_stddev>0.001</bias_stddev>
-              </noise>
-            </z>
-          </linear_acceleration>
-        </imu>
-      </sensor>
-    </gazebo>
-    <link name="${prefix}camera_link">
-      <visual>
-        <origin xyz="0 0 0" rpy="0 0 0"/>
-        <geometry>
-          <box size="0.015 0.130 0.022"/>
-        </geometry>
-      </visual>
-      <collision>
-        <origin xyz="0 0 0" rpy="0 0 0"/>
-        <geometry>
-          <box size="0.015 0.130 0.022"/>
-        </geometry>
-      </collision>
-      <inertial>
-        <origin xyz="0 0 0" rpy="0 0 0"/>
-        <mass value="0.035"/>
-        <inertia ixx="0.001"  ixy="0"  ixz="0" iyy="0.001" iyz="0" izz="0.001" />
-      </inertial>
-    </link>
-    <joint name="${prefix}camera_joint" type="fixed">
-      <parent link="${prefix}chassis"/>
-      <child link="${prefix}camera_link"/>
-      <origin xyz="0.215 0 0.05" rpy="0 0 0"/>
-    </joint>
-    <link name="${prefix}camera_depth_frame"/>
-    <joint name="${prefix}camera_depth_joint" type="fixed">
-      <origin xyz="0 0 0" rpy="${-pi/2} 0 ${-pi/2}"/>
-      <parent link="${prefix}camera_link"/>
-      <child link="${prefix}camera_depth_frame"/>
-    </joint>
-    <gazebo reference="${prefix}camera_link">
-      <sensor name="depth_camera" type="depth">
-        <visualize>true</visualize>
-        <update_rate>30.0</update_rate>
-        <camera name="camera">
-          <horizontal_fov>1.047198</horizontal_fov>
-          <image>
-            <width>640</width>
-            <height>480</height>
-            <format>R8G8B8</format>
-          </image>
-          <clip>
-            <near>0.05</near>
-            <far>3</far>
-          </clip>
-        </camera>
-        <plugin name="depth_camera_controller" filename="libgazebo_ros_camera.so">
-          <baseline>0.2</baseline>
-          <alwaysOn>true</alwaysOn>
-          <updateRate>0.0</updateRate>
-          <frame_name>camera_depth_frame</frame_name>
-          <pointCloudCutoff>0.5</pointCloudCutoff>
-          <pointCloudCutoffMax>3.0</pointCloudCutoffMax>
-          <distortionK1>0</distortionK1>
-          <distortionK2>0</distortionK2>
-          <distortionK3>0</distortionK3>
-          <distortionT1>0</distortionT1>
-          <distortionT2>0</distortionT2>
-          <CxPrime>0</CxPrime>
-          <Cx>0</Cx>
-          <Cy>0</Cy>
-          <focalLength>0</focalLength>
-          <hackBaseline>0</hackBaseline>
-        </plugin>
-      </sensor>
-    </gazebo>
   </xacro:macro>
 </robot>
