Commit message: functional effort controller for 4wd

File: psd_ws/install/psd_vehicle_description/share/psd_vehicle_description/urdf/psd_vehicle_macro.urdf.xacro (robot description, xacro)
@@ -1,297 +1 @@
-<?xml version="1.0" ?>
-<robot name="psd_vehicle" xmlns:xacro="http://www.ros.org/wiki/xacro">
-  <!-- include materials -->
-  <xacro:include filename="$(find psd_vehicle_description)/urdf/materials.xacro" />
-  <!-- start vehicle description -->
-  <xacro:macro name="psd_vehicle" params="prefix parent *origin">
-    <!-- LINKS -->
-    <!-- Chassis START-->
-    <link name="${prefix}chassis">
-      <inertial>
-        <origin xyz="-0.055282024534886974 0.006459558608433099 1.621642854614675e-05" rpy="0 0 0"/>
-        <mass value="7.077984465449566"/>
-        <inertia ixx="0.233109" iyy="0.053798" izz="0.264742" ixy="-0.0" iyz="-0.0" ixz="-0.0"/>
-      </inertial>
-      <visual>
-        <origin xyz="0 0 0" rpy="0 0 0"/>
-        <geometry>
-          <mesh filename="$(find psd_vehicle_description)/meshes/visual/base_link.stl" scale="0.001 0.001 0.001"/>
-        </geometry>
-        <material name="anodized_red"/>
-      </visual>
-      <collision>
-        <origin xyz="0 0 0" rpy="0 0 0"/>
-        <geometry>
-          <mesh filename="$(find psd_vehicle_description)/meshes/collision/base_link.stl" scale="0.001 0.001 0.001"/>
-        </geometry>
-      </collision>
-    </link>
-    <joint name="${prefix}world_joint" type="fixed">
-      <xacro:insert_block name="origin" />
-      <parent link="${parent}" />
-      <child link="${prefix}chassis" />
-    </joint>
-    <link name="${prefix}perno_FL_1">
-      <inertial>
-        <origin xyz="-0.000906687358749575 0.00042296243032097225 2.1642838935455414e-07" rpy="0 0 0"/>
-        <mass value="0.00011097676048806171"/>
-        <inertia ixx="0.0" iyy="0.0" izz="0.0" ixy="-0.0" iyz="0.0" ixz="-0.0"/>
-      </inertial>
-      <visual>
-        <origin xyz="0.230783 -0.306869 -1.6e-05" rpy="0 0 0"/>
-        <geometry>
-          <mesh filename="$(find psd_vehicle_description)/meshes/visual/perno_FL_1.stl" scale="0.001 0.001 0.001"/>
-        </geometry>
-        <material name="silver"/>
-      </visual>
-      <collision>
-        <origin xyz="0.230783 -0.306869 -1.6e-05" rpy="0 0 0"/>
-        <geometry>
-          <mesh filename="$(find psd_vehicle_description)/meshes/collision/perno_FL_1.stl" scale="0.001 0.001 0.001"/>
-        </geometry>
-      </collision>
-    </link>
-    <link name="${prefix}tyre_FL_1">
-      <inertial>
-        <origin xyz="-0.03851807609484373 0.017960856816041648 2.1642854673904234e-07" rpy="0 0 0"/>
-        <mass value="0.1944554118066591"/>
-        <inertia ixx="0.001191" iyy="0.000933" izz="0.000861" ixy="-0.000154" iyz="0.0" ixz="0.0"/>
-      </inertial>
-      <visual>
-        <origin xyz="0.232596 -0.307715 -1.6e-05" rpy="0 0 0"/>
-        <geometry>
-          <mesh filename="$(find psd_vehicle_description)/meshes/visual/tyre_FL_1.stl" scale="0.001 0.001 0.001"/>
-        </geometry>
-        <material name="rubber_tyre"/>
-      </visual>
-      <collision>
-        <origin xyz="0.232596 -0.307715 -1.6e-05" rpy="0 0 0"/>
-        <geometry>
-          <mesh filename="$(find psd_vehicle_description)/meshes/collision/tyre_FL_1.stl" scale="0.001 0.001 0.001"/>
-        </geometry>
-      </collision>
-    </link>z
-    <link name="${prefix}perno_FR_1">
-      <inertial>
-        <origin xyz="0.000905928215323884 -0.0004222740931605351 2.1642839664261197e-07" rpy="0 0 0"/>
-        <mass value="0.0001109767604880609"/>
-        <inertia ixx="0.0" iyy="0.0" izz="0.0" ixy="-0.0" iyz="-0.0" ixz="0.0"/>
-      </inertial>
-      <visual>
-        <origin xyz="-0.120217 -0.306869 -1.6e-05" rpy="0 0 0"/>
-        <geometry>
-          <mesh filename="$(find psd_vehicle_description)/meshes/visual/perno_FR_1.stl" scale="0.001 0.001 0.001"/>
-        </geometry>
-        <material name="silver"/>
-      </visual>
-      <collision>
-        <origin xyz="-0.120217 -0.306869 -1.6e-05" rpy="0 0 0"/>
-        <geometry>
-          <mesh filename="$(find psd_vehicle_description)/meshes/collision/perno_FR_1.stl" scale="0.001 0.001 0.001"/>
-        </geometry>
-      </collision>
-    </link>
-    <link name="${prefix}tyre_FR_1">
-      <inertial>
-        <origin xyz="0.03851831695141855 -0.017961168478880185 2.1642854608751476e-07" rpy="0 0 0"/>
-        <mass value="0.19445541180665865"/>
-        <inertia ixx="0.001191" iyy="0.000933" izz="0.000861" ixy="-0.000154" iyz="-0.0" ixz="0.0"/>
-      </inertial>
-      <visual>
-        <origin xyz="-0.122029 -0.306024 -1.6e-05" rpy="0 0 0"/>
-        <geometry>
-          <mesh filename="$(find psd_vehicle_description)/meshes/visual/tyre_FR_1.stl" scale="0.001 0.001 0.001"/>
-        </geometry>
-        <material name="rubber_tyre"/>
-      </visual>
-      <collision>
-        <origin xyz="-0.122029 -0.306024 -1.6e-05" rpy="0 0 0"/>
-        <geometry>
-          <mesh filename="$(find psd_vehicle_description)/meshes/collision/tyre_FR_1.stl" scale="0.001 0.001 0.001"/>
-        </geometry>
-      </collision>
-    </link>
-    <link name="${prefix}tyre_RR_1">
-      <inertial>
-        <origin xyz="0.04250016447333546 3.441685788030391e-07 2.16428546438244e-07" rpy="0 0 0"/>
-        <mass value="0.19445541180665948"/>
-        <inertia ixx="0.001262" iyy="0.000861" izz="0.000861" ixy="-0.0" iyz="-0.0" ixz="0.0"/>
-      </inertial>
-      <visual>
-        <origin xyz="-0.119284 0.293131 -1.6e-05" rpy="0 0 0"/>
-        <geometry>
-          <mesh filename="$(find psd_vehicle_description)/meshes/visual/tyre_RR_1.stl" scale="0.001 0.001 0.001"/>
-        </geometry>
-        <material name="rubber_tyre"/>
-      </visual>
-      <collision>
-        <origin xyz="-0.119284 0.293131 -1.6e-05" rpy="0 0 0"/>
-        <geometry>
-          <mesh filename="$(find psd_vehicle_description)/meshes/collision/tyre_RR_1.stl" scale="0.001 0.001 0.001"/>
-        </geometry>
-      </collision>
-    </link>
-    <link name="${prefix}link_RL_1">
-      <inertial>
-        <origin xyz="-0.047944553368047954 3.441685789140614e-07 2.1642854618965338e-07" rpy="0 0 0"/>
-        <mass value="0.09195911794645473"/>
-        <inertia ixx="6.5e-05" iyy="0.000142" izz="0.000206" ixy="-0.0" iyz="0.0" ixz="0.0"/>
-      </inertial>
-      <visual>
-        <origin xyz="0.095283 0.293131 -1.6e-05" rpy="0 0 0"/>
-        <geometry>
-          <mesh filename="$(find psd_vehicle_description)/meshes/visual/link_RL_1.stl" scale="0.001 0.001 0.001"/>
-        </geometry>
-        <material name="anodized_blue"/>
-      </visual>
-      <collision>
-        <origin xyz="0.095283 0.293131 -1.6e-05" rpy="0 0 0"/>
-        <geometry>
-          <mesh filename="$(find psd_vehicle_description)/meshes/collision/link_RL_1.stl" scale="0.001 0.001 0.001"/>
-        </geometry>
-      </collision>
-    </link>
-    <link name="${prefix}link_RR_1">
-      <inertial>
-        <origin xyz="0.04794379422462264 3.441685790250837e-07 2.1642854618632285e-07" rpy="0 0 0"/>
-        <mass value="0.09195911794645475"/>
-        <inertia ixx="6.5e-05" iyy="0.000142" izz="0.000206" ixy="0.0" iyz="-0.0" ixz="0.0"/>
-      </inertial>
-      <visual>
-        <origin xyz="0.015283 0.293131 -1.6e-05" rpy="0 0 0"/>
-        <geometry>
-          <mesh filename="$(find psd_vehicle_description)/meshes/visual/link_RR_1.stl" scale="0.001 0.001 0.001"/>
-        </geometry>
-        <material name="anodized_blue"/>
-      </visual>
-      <collision>
-        <origin xyz="0.015283 0.293131 -1.6e-05" rpy="0 0 0"/>
-        <geometry>
-          <mesh filename="$(find psd_vehicle_description)/meshes/collision/link_RR_1.stl" scale="0.001 0.001 0.001"/>
-        </geometry>
-      </collision>
-    </link>
-    <link name="${prefix}tyre_RL_1">
-      <inertial>
-        <origin xyz="-0.04249992361676111 3.4416857908059484e-07 2.1642854653184114e-07" rpy="0 0 0"/>
-        <mass value="0.19445541180665912"/>
-        <inertia ixx="0.001262" iyy="0.000861" izz="0.000861" ixy="0.0" iyz="0.0" ixz="0.0"/>
-      </inertial>
-      <visual>
-        <origin xyz="0.229851 0.293131 -1.6e-05" rpy="0 0 0"/>
-        <geometry>
-          <mesh filename="$(find psd_vehicle_description)/meshes/visual/tyre_RL_1.stl" scale="0.001 0.001 0.001"/>
-        </geometry>
-        <material name="rubber_tyre"/>
-      </visual>
-      <collision>
-        <origin xyz="0.229851 0.293131 -1.6e-05" rpy="0 0 0"/>
-        <geometry>
-          <mesh filename="$(find psd_vehicle_description)/meshes/collision/tyre_RL_1.stl" scale="0.001 0.001 0.001"/>
-        </geometry>
-      </collision>
-    </link>
-    <link name="${prefix}link_FL_1">
-      <inertial>
-        <origin xyz="-0.04795315128569644 3.441685794691729e-07 2.1642854620519813e-07" rpy="0 0 0"/>
-        <mass value="0.09196821373647668"/>
-        <inertia ixx="6.5e-05" iyy="0.000142" izz="0.000206" ixy="0.0" iyz="0.0" ixz="-0.0"/>
-      </inertial>
-      <visual>
-        <origin xyz="0.095283 -0.306869 -1.6e-05" rpy="0 0 0"/>
-        <geometry>
-          <mesh filename="$(find psd_vehicle_description)/meshes/visual/link_FL_1.stl" scale="0.001 0.001 0.001"/>
-        </geometry>
-        <material name="anodized_blue"/>
-      </visual>
-      <collision>
-        <origin xyz="0.095283 -0.306869 -1.6e-05" rpy="0 0 0"/>
-        <geometry>
-          <mesh filename="$(find psd_vehicle_description)/meshes/collision/link_FL_1.stl" scale="0.001 0.001 0.001"/>
-        </geometry>
-      </collision>
-    </link>
-    <link name="${prefix}link_FR_1">
-      <inertial>
-        <origin xyz="0.04795239214227047 3.441685796912175e-07 2.164285462018676e-07" rpy="0 0 0"/>
-        <mass value="0.09196821373647673"/>
-        <inertia ixx="6.5e-05" iyy="0.000142" izz="0.000206" ixy="-0.0" iyz="0.0" ixz="0.0"/>
-      </inertial>
-      <visual>
-        <origin xyz="0.015283 -0.306869 -1.6e-05" rpy="0 0 0"/>
-        <geometry>
-          <mesh filename="$(find psd_vehicle_description)/meshes/visual/link_FR_1.stl" scale="0.001 0.001 0.001"/>
-        </geometry>
-        <material name="anodized_blue"/>
-      </visual>
-      <collision>
-        <origin xyz="0.015283 -0.306869 -1.6e-05" rpy="0 0 0"/>
-        <geometry>
-          <mesh filename="$(find psd_vehicle_description)/meshes/collision/link_FR_1.stl" scale="0.001 0.001 0.001"/>
-        </geometry>
-      </collision>
-    </link>
-    <!-- JOINTS -->
-    <joint name="${prefix}steering_fl" type="revolute">
-      <origin xyz="-0.1355 0.0 0.0" rpy="0 0 0"/>
-      <parent link="${prefix}link_FL_1"/>
-      <child link="${prefix}perno_FL_1"/>
-      <axis xyz="0.0 -0.0 1.0"/>
-      <limit upper="0.523599" lower="-0.523599" effort="100" velocity="100"/>
-      <mimic joint="${prefix}steering_fr" multiplier="1.0" offset="0.0"/>
-    </joint>
-    <joint name="${prefix}drive_fl" type="continuous">
-      <origin xyz="-0.001813 0.000846 0.0" rpy="0 0 0"/>
-      <parent link="${prefix}perno_FL_1"/>
-      <child link="${prefix}tyre_FL_1"/>
-      <axis xyz="-0.906308 0.422618 0.0"/>
-      <mimic joint="${prefix}drive_rl" multiplier="1.0" offset="0.0"/>
-    </joint>
-    <joint name="${prefix}steering_fr" type="revolute">
-      <origin xyz="0.1355 0.0 0.0" rpy="0 0 0"/>
-      <parent link="${prefix}link_FR_1"/>
-      <child link="${prefix}perno_FR_1"/>
-      <axis xyz="0.0 -0.0 1.0"/>
-      <limit upper="0.523599" lower="-0.523599" effort="100" velocity="100"/>
-    </joint>
-    <joint name="${prefix}drive_fr" type="continuous">
-      <origin xyz="0.001812 -0.000845 0.0" rpy="0 0 0"/>
-      <parent link="${prefix}perno_FR_1"/>
-      <child link="${prefix}tyre_FR_1"/>
-      <axis xyz="0.906308 -0.422618 -0.0"/>
-      <mimic joint="${prefix}drive_rr" multiplier="1.0" offset="0.0"/>
-    </joint>
-    <joint name="${prefix}drive_rr" type="continuous">
-      <origin xyz="0.134567 0.0 0.0" rpy="0 0 0"/>
-      <parent link="${prefix}link_RR_1"/>
-      <child link="${prefix}tyre_RR_1"/>
-      <axis xyz="1.0 0.0 -0.0"/>
-    </joint>
-    <joint name="${prefix}suspension_rl" type="fixed">
-      <origin xyz="-0.095283 -0.293131 1.6e-05" rpy="0 0 0"/>
-      <parent link="${prefix}chassis"/>
-      <child link="${prefix}link_RL_1"/>
-    </joint>
-    <joint name="${prefix}suspension_rr" type="fixed">
-      <origin xyz="-0.015283 -0.293131 1.6e-05" rpy="0 0 0"/>
-      <parent link="${prefix}chassis"/>
-      <child link="${prefix}link_RR_1"/>
-    </joint>
-    <joint name="${prefix}drive_rl" type="continuous">
-      <origin xyz="-0.134568 0.0 0.0" rpy="0 0 0"/>
-      <parent link="${prefix}link_RL_1"/>
-      <child link="${prefix}tyre_RL_1"/>
-      <axis xyz="-1.0 -0.0 0.0"/>
-    </joint>
-    <joint name="${prefix}suspension_fl" type="fixed">
-      <origin xyz="-0.095283 0.306869 1.6e-05" rpy="0 0 0"/>
-      <parent link="${prefix}chassis"/>
-      <child link="${prefix}link_FL_1"/>
-    </joint>
-    <joint name="${prefix}suspension_fr" type="fixed">
-      <origin xyz="-0.015283 0.306869 1.6e-05" rpy="0 0 0"/>
-      <parent link="${prefix}chassis"/>
-      <child link="${prefix}link_FR_1"/>
-    </joint>
-  </xacro:macro>
-</robot>
+/home/ubuntu/psd_ws/src/psd_vehicle_description/urdf/psd_vehicle_macro.urdf.xacro

File: psd_ws/src/psd_vehicle_description/urdf/psd_vehicle.urdf.xacro (robot description, xacro)
@@ -1,18 +1,14 @@
 <?xml version="1.0" encoding="UTF-8"?>
 <robot xmlns:xacro="http://wiki.ros.org/xacro" name="psd_vehicle">
-  <!-- Use this if parameters are set from the launch file, otherwise delete -->
-  <xacro:arg name="prefix" default="" />
-  <xacro:arg name="simulation_controllers" default="" />
   <xacro:include filename="$(find psd_vehicle_description)/urdf/psd_vehicle_macro.urdf.xacro"/>
   <xacro:include filename="$(find psd_vehicle_description)/urdf/psd_vehicle_macro.ros2_control.xacro"/>
   <!-- Load robot's macro with parameters -->
-  <link name="leo" />
+  <link name="home" />
   <!-- set prefix if multiple robots are used -->
-  <xacro:psd_vehicle prefix="$(arg prefix)" parent="leo" >
+  <xacro:psd_vehicle parent="home" >
     <origin xyz="0 0 0.095" rpy="0 0 0" />          <!-- position robot in the world -->
   </xacro:psd_vehicle>
   <xacro:psd_vehicle_ros2_control
     name="psd_vehicle"
-    prefix="$(arg prefix)"
   />
 </robot>

File: psd_ws/src/psd_vehicle_description/urdf/psd_vehicle_macro.ros2_control.xacro (robot description, xacro)
@@ -2,67 +2,77 @@
 <robot xmlns:xacro="http://wiki.ros.org/xacro">
   <xacro:macro name="psd_vehicle_ros2_control" params="
-                name
-                prefix
-                use_mock_hardware:=^|false
-                mock_sensor_commands:=^|false
-                sim_gazebo:=^|false"
+                name"
                 >
-    <ros2_control name="${name}" type="system">
+    <!-- control -->
+    <xacro:property name="PI" value="3.14159265359" />
+    <xacro:property name="max_torque" value="100" />
+    <xacro:property name="max_steering_angle" value="${20 * PI / 180}" />
+    <ros2_control name="GazeboSimSystem" type="system">
       <hardware>
-        <xacro:if value="${use_mock_hardware}">
-          <plugin>mock_components/GenericSystem</plugin>
-          <param name="mock_sensor_commands">${mock_sensor_commands}</param>
-        </xacro:if>
-        <xacro:if value="${sim_gazebo}">
-          <plugin>ign_ros2_control/IgnitionSystem</plugin>
-        </xacro:if>
+        <plugin>gz_ros2_control/GazeboSimSystem</plugin>
       </hardware>
-      <joint name="${prefix}steering_fl">
-        <command_interface name="position"/>
-        <state_interface name="position"/>
+      <!-- steering control -->
+      <joint name="steering_fr">
+        <command_interface name="position">
+          <param name="min">"${-max_steering_angle}"</param>
+          <param name="max">"${max_steering_angle}"</param>
+        </command_interface>
+        <state_interface name="position">
+          <param name="initial_value">0.0</param>
+        </state_interface>
       </joint>
-      <joint name="${prefix}steering_fr">
-        <command_interface name="position"/>
-        <state_interface name="position"/>
+      <joint name="steering_fl">
+        <command_interface name="position">
+          <param name="min">"${-max_steering_angle}"</param>
+          <param name="max">"${max_steering_angle}"</param>
+        </command_interface>
+        <state_interface name="position">
+          <param name="initial_value">0.0</param>
+        </state_interface>
       </joint>
-      <joint name="${prefix}drive_rl">
-        <command_interface name="effort"/>
+      <!-- driving control -->
+      <joint name="drive_rl">
+        <command_interface name="effort">
+          <param name="min">"${-max_torque}"</param>
+          <param name="max">"${max_torque}"</param>
+        </command_interface>
         <state_interface name="position"/>
         <state_interface name="velocity"/>
+        <state_interface name="effort"/>
       </joint>
-      <joint name="${prefix}drive_rr">
-        <command_interface name="effort"/>
+      <joint name="drive_rr">
+        <command_interface name="effort">
+          <param name="min">"${-max_torque}"</param>
+          <param name="max">"${max_torque}"</param>
+        </command_interface>
         <state_interface name="position"/>
         <state_interface name="velocity"/>
+        <state_interface name="effort"/>
       </joint>
-      <joint name="${prefix}drive_fl">
-        <command_interface name="effort"/>
+      <joint name="drive_fl">
+        <command_interface name="effort">
+          <param name="min">"${-max_torque}"</param>
+          <param name="max">"${max_torque}"</param>
+        </command_interface>
         <state_interface name="position"/>
         <state_interface name="velocity"/>
+        <state_interface name="effort"/>
       </joint>
-      <joint name="${prefix}drive_fr">
-        <command_interface name="effort"/>
+      <joint name="drive_fr">
+        <command_interface name="effort">
+          <param name="min">"${-max_torque}"</param>
+          <param name="max">"${max_torque}"</param>
+        </command_interface>
         <state_interface name="position"/>
         <state_interface name="velocity"/>
+        <state_interface name="effort"/>
       </joint>
-      <sensor name="tcp_fts_sensor1">
-        <state_interface name="fx"/>
-        <state_interface name="fy"/>
-        <state_interface name="fz"/>
-        <state_interface name="tx"/>
-        <state_interface name="ty"/>
-        <state_interface name="tz"/>
-        <param name="frame_id">tyre_RL_1</param>
-      </sensor>
-      <sensor name="tcp_fts_sensor2">
-        <state_interface name="fx"/>
-        <state_interface name="fy"/>
-        <state_interface name="fz"/>
-        <state_interface name="tx"/>
-        <state_interface name="ty"/>
-        <state_interface name="tz"/>
-        <param name="frame_id">tyre_RR_1</param>
-      </sensor>
     </ros2_control>
+    <gazebo>
+      <!-- Joint state publisher -->
+      <plugin filename="gz_ros2_control-system" name="gz_ros2_control::GazeboSimROS2ControlPlugin">
+        <parameters>$(find psd_vehicle_bringup)/config/psd_vehicle_controllers.yaml</parameters>
+      </plugin>
+    </gazebo>
   </xacro:macro>
 </robot>
